File: Hardware/BoverJR.kicad_sch (KiCad schematic)
At the start: 27 parts, among them J1 HC_SRO4, J10 BOTON, J11 Alimentacion, J2 HC_SRO4, J3 HC_SRO4, J5 SWITCH, J7 Programador, J9 KY_032, U1 ESP32-WROOM-32, U2 L7805

Commit message: lo organize mejor
Parts:
- C2, C3: value 220uF -> (none)
- J4: value (none) -> Input of Driver L9110
- J6: value (none) -> Encoder de motores; footprint (none) -> EESTN5:pin_strip_4
- U?: value (none) -> LM1117-3.3
Other:
- note added: "Buttons"
- note added: "Conversor USB a UART"
- note added: "Encoder contador de vueltas para motores"
- moved on the sheet: J10, J6, J7
