File: Hardware/BoverOrogin_V2.kicad_pcb (KiCad board)
At the start: 2 copper layers, 100 x 100 mm, 24 parts, among them J1 DRV8833_OUT, J2 DRV8833_IN, J3 Encoder Derecho, J4 Encoder Izquierdo, J5 Distancia_Der, J6 Distancia_Izq, J7 Distancia_Frontal, J8 Conn_01x02, SW1 SW_Push, SW2 SW_SPDT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

Commit message: placa bover terminada, sensores acomodados
Parts:
- moved J6 16.3 mm to (126.0, 44.1)
- moved J7 9.13 mm to (145.1, 44.1)
- moved J5 8.81 mm to (165.0, 44.1), turned to -90 degrees
Connections:
- J5 pad 1: /IR_IZQ -> GND
- J5 pad 3: GND -> /IR_IZQ
Routing:
- net +5V: track 255.5 -> 283.6 mm
- net /IR_DER: track 6.61 -> 21.1 mm
- net /IR_FRONTAL: track 6.94 -> 16.2 mm
- net /IR_IZQ: track 7.53 -> 14.9 mm
- net GND: track 10.4 -> 15.5 mm, vias 4 -> 6
Changed lines of the file:
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@@
   (net 40 "unconnected-(U4-INT-Pad8)")
   (footprint "Connector_JST:JST_EH_B3B-EH-A_1x03_P2.50mm_Vertical" (layer "F.Cu")
-    (at 159.86 51.28 90)
+    (at 165 44.13 -90)
     (descr "JST EH series connector, B3B-EH-A (http://www.jst-mfg.com/product/pdf/eng/eEH.pdf), generated with kicad-footprint-generator")
     (tags "connector JST EH vertical")
@@
     (property "ki_keywords" "connector")
     (attr through_hole)
-    (fp_text reference "J5" (at 2.5 -2.8 90) (layer "F.SilkS")
+    (fp_text reference "J5" (at 2.53 -6.86 90) (layer "F.SilkS")
         (effects (font (size 1 1) (thickness 0.15)))
     )
@@
     (fp_line (start 7.5 2.2) (end 7.5 -1.6)
       (stroke (width 0.1) (type solid)) (layer "F.Fab"))
-    (pad "1" thru_hole roundrect (at 0 0 90) (size 1.7 1.95) (drill 0.95) (layers "*.Cu" "*.Mask") (roundrect_rratio 0.147059)
-      (net 20 "/IR_IZQ") (pinfunction "Pin_1") (pintype "passive"))
-    (pad "2" thru_hole oval (at 2.5 0 90) (size 1.7 1.95) (drill 0.95) (layers "*.Cu" "*.Mask")
+    (pad "1" thru_hole roundrect (at 0 0 270) (size 1.7 1.95) (drill 0.95) (layers "*.Cu" "*.Mask") (roundrect_rratio 0.147059)
+      (net 2 "GND") (pinfunction "Pin_1") (pintype "passive"))
+    (pad "2" thru_hole oval (at 2.5 0 270) (size 1.7 1.95) (drill 0.95) (layers "*.Cu" "*.Mask")
       (net 3 "+5V") (pinfunction "Pin_2") (pintype "passive"))
-    (pad "3" thru_hole oval (at 5 0 90) (size 1.7 1.95) (drill 0.95) (layers "*.Cu" "*.Mask")
-      (net 2 "GND") (pinfunction "Pin_3") (pintype "passive"))
+    (pad "3" thru_hole oval (at 5 0 270) (size 1.7 1.95) (drill 0.95) (layers "*.Cu" "*.Mask")
+      (net 20 "/IR_IZQ") (pinfunction "Pin_3") (pintype "passive"))
     (model "${KICAD6_3DMODEL_DIR}/Connector_JST.3dshapes/JST_EH_B3B-EH-A_1x03_P2.50mm_Vertical.wrl"
       (offset (xyz 0 0 0))
@@
   )
   (footprint "Connector_JST:JST_EH_B3B-EH-A_1x03_P2.50mm_Vertical" (layer "F.Cu")
-    (at 142.2 46.2 -90)
+    (at 126 44.1 -90)
     (descr "JST EH series connector, B3B-EH-A (http://www.jst-mfg.com/product/pdf/eng/eEH.pdf), generated with kicad-footprint-generator")
     (tags "connector JST EH vertical")
@@
   )
   (footprint "Connector_JST:JST_EH_B3B-EH-A_1x03_P2.50mm_Vertical" (layer "F.Cu")
-    (at 153.98 46.23 -90)
+    (at 145.1 44.1 -90)
     (descr "JST EH series connector, B3B-EH-A (http://www.jst-mfg.com/product/pdf/eng/eEH.pdf), generated with kicad-footprint-generator")
     (tags "connector JST EH vertical")
@@
     (style (thickness 0.1) (arrow_length 1.27) (text_position_mode 0) (extension_height 0.58642) (extension_offset 0.5) keep_text_aligned)
   )
-  (dimension (type aligned) (layer "Dwgs.User")
-    (pts (xy 146.879443 34.82) (xy 146.879443 134.82))
-    (height -66.03)
-    (gr_text "100,0000 mm" (at 211.759443 84.82 90) (layer "Dwgs.User")
-      (effects (font (size 1 1) (thickness 0.15)))
-    )
-    (format (prefix "") (suffix "") (units 3) (units_format 1) (precision 4))
-    (style (thickness 0.1) (arrow_length 1.27) (text_position_mode 0) (extension_height 0.58642) (extension_offset 0.5) keep_text_aligned)
-  )
   (dimension (type aligned) (layer "Edge.Cuts")
     (pts (xy 95 110) (xy 110 110))
@@
   (segment (start 134.58 61.27) (end 134.62 61.31) (width 1) (layer "F.Cu") (net 2))
   (segment (start 129.44 61.27) (end 134.58 61.27) (width 1) (layer "F.Cu") (net 2))
+  (segment (start 123.4 75.89) (end 123.4 70.75) (width 1) (layer "F.Cu") (net 2))
   (via (at 146 76.5) (size 1.5) (drill 1) (layers "F.Cu" "B.Cu") (free) (net 2))
   (via (at 129.44 61.27) (size 1.5) (drill 1) (layers "F.Cu" "B.Cu") (free) (net 2))
   (via (at 134.62 61.31) (size 1.5) (drill 1) (layers "F.Cu" "B.Cu") (free) (net 2))
+  (via (at 123.4 70.75) (size 1.5) (drill 1) (layers "F.Cu" "B.Cu") (free) (net 2))
+  (via (at 123.45 75.95) (size 1.5) (drill 1) (layers "F.Cu" "B.Cu") (free) (net 2))
   (via (at 140.82 76.46) (size 1.5) (drill 1) (layers "F.Cu" "B.Cu") (free) (net 2))
+  (segment (start 132.025 57.8) (end 132.025 55.625) (width 1) (layer "B.Cu") (net 3))
   (segment (start 132.025 63.95) (end 132.075 63.9) (width 1) (layer "B.Cu") (net 3))
-  (segment (start 134.3 48.7) (end 142.2 48.7) (width 1) (layer "B.Cu") (net 3))
-  (segment (start 142.2 48.7) (end 153.95 48.7) (width 1) (layer "B.Cu") (net 3))
+  (segment (start 132.025 55.625) (end 130.8 54.4) (width 1) (layer "B.Cu") (net 3))
   (segment (start 118.097 82.953) (end 118.097 81.05) (width 1) (layer "B.Cu") (net 3))
   (segment (start 119.9 78.35) (end 120.4 78.85) (width 1) (layer "B.Cu") (net 3))
+  (segment (start 126 46.6) (end 145.1 46.6) (width 1) (layer "B.Cu") (net 3))
   (segment (start 132.025 66.275) (end 132.025 63.95) (width 1) (layer "B.Cu") (net 3))
-  (segment (start 153.95 48.7) (end 153.98 48.73) (width 1) (layer "B.Cu") (net 3))
+  (segment (start 120.8 48.2) (end 122.4 46.6) (width 1) (layer "B.Cu") (net 3))
   (segment (start 129.42 70.42) (end 128.65 69.65) (width 1) (layer "B.Cu") (net 3))
   (segment (start 102.855 75.25) (end 118.047 75.25) (width 1) (layer "B.Cu") (net 3))
+  (segment (start 164.97 46.6) (end 165 46.63) (width 1) (layer "B.Cu") (net 3))
   (segment (start 118.097 74.353) (end 118.825 73.625) (width 1) (layer "B.Cu") (net 3))
+  (segment (start 130.8 54.4) (end 122.8 54.4) (width 1) (layer "B.Cu") (net 3))
   (segment (start 118.097 78.35) (end 119.9 78.35) (width 1) (layer "B.Cu") (net 3))
   (segment (start 118.097 75.3) (end 118.097 74.353) (width 1) (layer "B.Cu") (net 3))
@@
   (segment (start 132.075 63.9) (end 136.553 63.9) (width 1) (layer "B.Cu") (net 3))
   (segment (start 134.12 97.62) (end 136.73 100.23) (width 1) (layer "B.Cu") (net 3))
-  (segment (start 153.98 48.73) (end 159.81 48.73) (width 1) (layer "B.Cu") (net 3))
+  (segment (start 122.4 46.6) (end 126 46.6) (width 1) (layer "B.Cu") (net 3))
+  (segment (start 122.8 54.4) (end 120.8 52.4) (width 1) (layer "B.Cu") (net 3))
   (segment (start 118.825 73.625) (end 119.35 73.1) (width 1) (layer "B.Cu") (net 3))
   (segment (start 125.2 73.1) (end 128.65 69.65) (width 1) (layer "B.Cu") (net 3))
@@
   (segment (start 120.4 78.85) (end 120.4 94.45) (width 1) (layer "B.Cu") (net 3))
   (segment (start 169.5 100.52) (end 169.5 102.72) (width 1) (layer "B.Cu") (net 3))
-  (segment (start 132.025 50.975) (end 134.3 48.7) (width 1) (layer "B.Cu") (net 3))
   (segment (start 136.55 67.85) (end 136.553 67.847) (width 1) (layer "B.Cu") (net 3))
   (segment (start 149.85 68.497) (end 137.197 68.497) (width 1) (layer "B.Cu") (net 3))
@@
   (segment (start 134.12 93.65) (end 134.12 97.62) (width 1) (layer "B.Cu") (net 3))
   (segment (start 120.4 94.45) (end 118 96.85) (width 1) (layer "B.Cu") (net 3))
-  (segment (start 132.025 57.8) (end 132.025 50.975) (width 1) (layer "B.Cu") (net 3))
   (segment (start 119.35 73.1) (end 125.2 73.1) (width 1) (layer "B.Cu") (net 3))
   (segment (start 118.097 78.35) (end 118.097 75.3) (width 1) (layer "B.Cu") (net 3))
@@
   (segment (start 117.6 83.45) (end 118.097 82.953) (width 1) (layer "B.Cu") (net 3))
   (segment (start 169.21 100.23) (end 169.5 100.52) (width 1) (layer "B.Cu") (net 3))
-  (segment (start 159.81 48.73) (end 159.86 48.78) (width 1) (layer "B.Cu") (net 3))
+  (segment (start 120.8 52.4) (end 120.8 48.2) (width 1) (layer "B.Cu") (net 3))
   (segment (start 128.65 69.65) (end 132.025 66.275) (width 1) (layer "B.Cu") (net 3))
   (segment (start 143.45 70.42) (end 143.45 84.32) (width 1) (layer "B.Cu") (net 3))
+  (segment (start 145.1 46.6) (end 164.97 46.6) (width 1) (layer "B.Cu") (net 3))
   (segment (start 118.097 78.35) (end 118.097 81.05) (width 1) (layer "B.Cu") (net 3))
   (segment (start 117.6 84.8) (end 117.6 83.45) (width 1) (layer "B.Cu") (net 3))
@@
   (segment (start 152.345 60.395) (end 159 67.05) (width 0.75) (layer "B.Cu") (net 19))
   (segment (start 180.5 91.05) (end 174.5 97.05) (width 0.75) (layer "B.Cu") (net 19))
-  (segment (start 157.425 56.135) (end 159.86 53.7) (width 0.75) (layer "B.Cu") (net 20))
-  (segment (start 159.86 53.7) (end 159.86 51.28) (width 0.75) (layer "B.Cu") (net 20))
-  (segment (start 157.425 57.8) (end 157.425 56.135) (width 0.75) (layer "B.Cu") (net 20))
-  (segment (start 142.2 51.2) (end 142.2 57.785) (width 0.75) (layer "B.Cu") (net 21))
-  (segment (start 142.2 57.785) (end 142.185 57.8) (width 0.75) (layer "B.Cu") (net 21))
-  (segment (start 154.885 56.055) (end 153.98 55.15) (width 0.75) (layer "B.Cu") (net 22))
-  (segment (start 154.885 57.8) (end 154.885 56.055) (width 0.75) (layer "B.Cu") (net 22))
-  (segment (start 153.98 55.15) (end 153.98 51.23) (width 0.75) (layer "B.Cu") (net 22))
+  (segment (start 159.67 49.13) (end 165 49.13) (width 0.75) (layer "B.Cu") (net 20))
+  (segment (start 157.425 51.375) (end 159.67 49.13) (width 0.75) (layer "B.Cu") (net 20))
+  (segment (start 157.425 57.8) (end 157.425 51.375) (width 0.75) (layer "B.Cu") (net 20))
+  (segment (start 135.7 49.1) (end 126 49.1) (width 0.75) (layer "B.Cu") (net 21))
+  (segment (start 142.185 55.585) (end 135.7 49.1) (width 0.75) (layer "B.Cu") (net 21))
+  (segment (start 142.185 57.8) (end 142.185 55.585) (width 0.75) (layer "B.Cu") (net 21))
+  (segment (start 154.885 53.085) (end 150.9 49.1) (width 0.75) (layer "B.Cu") (net 22))
+  (segment (start 150.9 49.1) (end 145.1 49.1) (width 0.75) (layer "B.Cu") (net 22))
+  (segment (start 154.885 57.8) (end 154.885 53.085) (width 0.75) (layer "B.Cu") (net 22))
   (segment (start 100.95 75.25) (end 100.95 78.28) (width 0.75) (layer "B.Cu") (net 23))
   (segment (start 100.95 78.28) (end 101.05 78.38) (width 0.75) (layer "B.Cu") (net 23))
