File: Hardware/BoverOrogin_V2.kicad_sch (KiCad schematic)
At the start: 25 parts, among them J1 DRV8833_OUT, J2 DRV8833_IN, J3 Encoder Derecho, J4 Encoder Izquierdo, J5 Distancia_Der, J6 Distancia_Izq, J7 Distancia_Frontal, J8 Conn_01x02, SW1 SW_Push, SW2 SW_SPDT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

Commit message: placa bover terminada, sensores acomodados
Connections:
- net GND: now also J5.1 (Pin_1); no longer J5.3 (Pin_3)
- net IR_IZQ: now also J5.3 (Pin_3); no longer J5.1 (Pin_1)
Changed lines of the file:
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@@
     (stroke (width 0) (type default))
   )
-  (wire (pts (xy 196.85 154.94) (xy 187.198 154.94))
+  (wire (pts (xy 196.85 149.86) (xy 187.198 149.86))
     (stroke (width 0) (type default))
   )
@@
     (stroke (width 0) (type default))
   )
-  (wire (pts (xy 187.198 154.94) (xy 187.198 156.718))
+  (wire (pts (xy 187.198 149.86) (xy 187.198 151.638))
     (stroke (width 0) (type default))
   )
@@
     (effects (font (size 1.27 1.27)) (justify right bottom))
   )
-  (label "IR_IZQ" (at 196.85 149.86 180) (fields_autoplaced)
+  (label "IR_IZQ" (at 196.85 154.94 180) (fields_autoplaced)
     (effects (font (size 1.27 1.27)) (justify right bottom))
   )
@@
     )
   )
-  (symbol (lib_id "power:GND") (at 187.198 156.718 0) (unit 1)
+  (symbol (lib_id "power:GND") (at 187.198 151.638 0) (unit 1)
     (in_bom yes) (on_board yes) (dnp no)
-    (property "Reference" "#PWR019" (at 187.198 163.068 0)
+    (property "Reference" "#PWR019" (at 187.198 157.988 0)
       (effects (font (size 1.27 1.27)) hide)
     )
-    (property "Value" "GND" (at 187.198 161.29 0)
+    (property "Value" "GND" (at 187.198 156.21 0)
       (effects (font (size 1.27 1.27)))
     )
-    (property "Footprint" "" (at 187.198 156.718 0)
+    (property "Footprint" "" (at 187.198 151.638 0)
       (effects (font (size 1.27 1.27)) hide)
     )
-    (property "Datasheet" "" (at 187.198 156.718 0)
+    (property "Datasheet" "" (at 187.198 151.638 0)
       (effects (font (size 1.27 1.27)) hide)
     )
