File: Hardware/BoverJr_embebido/BoverJr_embebido/BoverJr_embebido.kicad_sch (KiCad schematic)
At the start: 35 parts, among them J1 DRV8833_OUT, J2 DRV8833_IN, J3 Encoder Derecho, J4 Encoder Izquierdo, J5 Distancia_Der, J6 Distancia_Izq, J7 Distancia_Frontal, J8 Conn_01x02, J9 uart, SW1 SW_Push, SW2 SW_SPDT, SW3 SW_Push, U1 L7805, U3 QRE1113, U4 GY-521, U6 ESP32-WROOM-32, U7 AMS1117-3.3

Commit message: Placa Flecha Verde terminada
Parts:
- removed C7, C8: C, symbol Device:C
- removed J1: DRV8833_OUT, Connector_PinSocket_2.54mm:PinSocket_1x06_P2.54mm_Vertical, symbol Connector_Generic:Conn_01x06
- removed J2: DRV8833_IN, Connector_PinSocket_2.54mm:PinSocket_1x06_P2.54mm_Vertical, symbol Connector_Generic:Conn_01x06
- removed J9: uart, symbol Connector_Generic_MountingPin:Conn_01x03_MountingPin
- removed R1: 100, EESTN5:R_1206, symbol EESTN5:R
- removed R2: 10K, EESTN5:R_1206, symbol EESTN5:R
- removed U3: QRE1113, EESTN5:QRE1113GR, symbol EESTN5:QRE1113
- removed U6: ESP32-WROOM-32, chip2:Chipesp32, symbol ESP32-WROOM-32:ESP32-WROOM-32
- added J9: UART, EESTN5:Pin_Header_3, symbol EESTN5:CONN_01X03
- added U1: ESP32-WROOM-32E, ESP32-WROOM-32E:ESP32-WROOM-32E, symbol ESP32-WROOM-32E:ESP32-WROOM-32E
- added U5: DRV8833, EESTN5:HTSSOP-16, symbol EESTN5:DRV8833
- C10, C5, C6, C9: footprint (none) -> EESTN5:C_1206
- J8: value Conn_01x02 -> IN
- LED1: footprint EESTN5:led_3mm_clear -> EESTN5:Led_0805
- R4: footprint (none) -> EESTN5:R_1206
- SW2: footprint EESTN5:SW_SPDT_TH_Vertical -> Button_Switch_THT:SW_Slide_1P2T_CK_OS102011MS2Q
- SW_BOOT1: renamed from SW3; footprint (none) -> EESTN5:PUSH_SWITCH_THT
- U4: value GY-521 -> MPU
Connections:
- net +3.3V: now also U1.2 (VDD)
- net +BATT: now also U5.14 (VINT)
- net AIN1: now also U1.19 (NC@19), U5.16 (AIN1)
- net AIN2: now also U1.20 (NC@20), U5.15 (AIN2)
- net AOUT1: now also U5.2 (AOUT1)
- net AOUT2: now also U5.4 (AOUT2)
- net BIN1: now also U1.22 (NC@22), U5.9 (BIN1)
- net BIN2: now also U1.21 (NC@21), U5.10 (BIN2)
- net BOOT: now also U1.25 (IO0)
- net BOUT1: now also U5.7 (BOUT1)
- net BOUT2: now also U5.5 (BOUT2)
- net D1A: now also U1.18 (NC@18)
- net D1B: now also U1.11 (IO26)
- net D2A: now also J4.5 (Pin_5), U1.30 (IO18); no longer J4.4 (Pin_4)
- net D2B: now also J4.4 (Pin_4), U1.29 (IO5); no longer J4.5 (Pin_5)
- net EN: now also U1.3 (EN)
- net GND: now also J9.3 (P3), U1.1 (GND@1), U1.15 (GND@15), U1.38 (GND@38), U1.GND@39 (THERMAL@39), U1.GND@40 (THERMAL@39), U1.GND@41 (THERMAL@39), U1.GND@42 (THERMAL@39), U1.GND@43 (THERMAL@39), U1.GND@44 (THERMAL@39), U1.GND@45 (THERMAL@39), U1.GND@46 (THERMAL@39), U1.GND@47 (THERMAL@39), U5.13 (GND)
- net IR_DER: now also U1.12 (IO27)
- net IR_FRONTAL: now also U1.6 (IO34)
- net IR_IZQ: now also U1.7 (IO35)
- net RX: now also J9.2 (P2), U1.34 (IO3)
- net SCL: now also U1.17 (NC@17)
- net SDA: now also U1.16 (IO13)
- net TX: now also J9.1 (P1), U1.35 (IO1)
- net start: now also U1.10 (IO25)
- no-connect marks 1 -> 0
Other:
- note added: "Esp32"
- note removed: "Sensor Tatami"
- moved on the sheet: C9
