File: Hardware/Placas Embebidas/Flecha verde/Flecha_Verde_V1.kicad_pcb (KiCad board)
At the start: 2 copper layers, 100 x 90 mm, 28 parts, among them J1 Encoder Derecho, J2 Encoder Izquierdo, J3 IN, J4 Distancia_Der, J5 Distancia_Izq, J8 Distancia_Frontal, J9 UART, U1 ESP32-WROOM-32E, U2 MPU, U4 L7805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

Commit message: Placa terminada
Parts:
- removed J9: UART, EESTN5:Pin_Header_3
- removed LED1: 2V, EESTN5:Led_0805
- removed LLAVE1: SW_SPDT, Button_Switch_THT:SW_Slide_1P2T_CK_OS102011MS2Q
- added C11: 10nF, EESTN5:C_1206, F.Cu at (152.9, 90.7)
- added C12: 2,2uF, EESTN5:C_1206, F.Cu at (146.5, 90.7)
- added C13: 10uF, EESTN5:C_1206, F.Cu at (150.2, 90.7)
- added C7: 10uF, EESTN5:C_1206, F.Cu at (135.7, 86.5)
- added C8: 10uF, EESTN5:C_1206, F.Cu at (133.4, 74.4)
- added G***: LOGO, EESTN5:logo_fle2, F.Cu at (150.1, 118.8)
- added G***: LOGO, EESTN5:logo_fle, F.Cu at (150.4, 118.3)
- added J199: 7.4v, Connector_JST:JST_EH_B2B-EH-A_1x02_P2.50mm_Vertical, F.Cu at (109.5, 97.4)
- added J299: Jumper, EESTN5:SW_SPDT_TH_Vertical, F.Cu at (110.5, 87.3)
- added LED_ESP32: 2V, EESTN5:Led_0805, F.Cu at (132.0, 68.4)
- added R1: 470, EESTN5:R_0805, F.Cu at (134.8, 68.3)
- added R2: 10K, EESTN5:R_1206, F.Cu at (185.6, 81.5)
- added R5: 10K, EESTN5:R_1206, F.Cu at (156.8, 82.5)
- C1: value 220uF -> 10uF; moved to F.Cu
- C10, C2, C3, C4, J1, J2, J4, J5, J8, SW_START1, U1, U4, U5, U7: moved to F.Cu
- C5, C6, C9: value C -> 100nF; moved to F.Cu
- J3: value IN -> CP2102; footprint Connector_JST:JST_EH_B2B-EH-A_1x02_P2.50mm_Vertical -> EESTN5:Pin_Header_5; moved to F.Cu
- R3: value 470 -> 47K; footprint EESTN5:R_0805 -> EESTN5:R_1206; moved to F.Cu
- R4: value R -> 10k; moved to F.Cu
- SW_BOOT1: footprint EESTN5:PUSH_SWITCH_THT -> EESTN5:SW_SPST_EVQPE1; moved to F.Cu
- moved J3 73.6 mm to (180.4, 70.8), turned to -54 degrees
- moved J5 42.6 mm to (127.1, 61.5), turned to 54 degrees
- moved J4 42.6 mm to (170.1, 57.4), turned to -54 degrees
- moved C9 30.0 mm to (135.2, 57.7)
- moved R3 26.4 mm to (146.0, 101.6)
- moved SW_BOOT1 26.0 mm to (154.0, 77.9)
- moved R4 25.4 mm to (138.0, 57.7), turned to 90 degrees
- moved C5 15.8 mm to (135.7, 89.3)
- moved J2 12.6 mm to (118.1, 97.4), turned to 0 degrees
- moved C10 11.5 mm to (148.4, 79.3), turned to 90 degrees
- moved C6 11.1 mm to (133.4, 71.7), turned to 0 degrees
- moved U4 10.9 mm to (123.7, 80.2)
- moved U5 10.6 mm to (150.5, 99.8), turned to 0 degrees
- moved C2 9.29 mm to (122.8, 89.3), turned to 180 degrees
- moved C3 8.74 mm to (129.8, 87.9), turned to 90 degrees
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Connections:
- net /D2A renamed /OUT_M2_DB
- C5 pad 1: +5V -> +BATT
- J1 pad 1: /AOUT1 -> /OUT_A_MOTOR1
- J1 pad 2: /AOUT2 -> /OUT_B_MOTOR1
- J1 pad 3: +5V -> +3.3V
- J1 pad 4: /D1A -> /OUT_M1_DA
- J1 pad 5: /D1B -> /OUT_M1_DB
- J2 pad 1: /BOUT2 -> /OUT_A_MOTOR2
- J2 pad 2: /BOUT1 -> /OUT_B_MOTOR2
- J2 pad 3: +5V -> +3.3V
- J2 pad 4: /D2B -> /OUT_M2_DA
- J3 pad 1: GND -> /TX
- J3 pad 2: +BATT -> /RX
- R3 pad 1: Net-(LED1-A) -> +3.3V
- R3 pad 2: +5V -> Net-(U5-nSLEEP)
- SW_START1 pad 2: /start -> /START
- U1 pad 10: /start -> /M2_IN2
- U1 pad 11: /D1B -> /M1_IN2
- U1 pad 12: /IR_DER -> /M1_IN1
- U1 pad 16: /SDA -> unconnected-(U1-IO13-Pad16)
- U1 pad 17: /SCL -> unconnected-(U1-NC@17-Pad17)
- U1 pad 18: /D1A -> unconnected-(U1-NC@18-Pad18)
- U1 pad 19: /AIN1 -> unconnected-(U1-NC@19-Pad19)
- U1 pad 20: /AIN2 -> unconnected-(U1-NC@20-Pad20)
- U1 pad 21: /BIN2 -> unconnected-(U1-NC@21-Pad21)
- U1 pad 22: /BIN1 -> unconnected-(U1-NC@22-Pad22)
- U1 pad 26: unconnected-(U1-IO4-Pad26) -> /OUT_M1_DB
- U1 pad 27: unconnected-(U1-IO16-Pad27) -> /OUT_M1_DA
- U1 pad 28: unconnected-(U1-IO17-Pad28) -> /IR_IZQ
- U1 pad 29: /D2B -> unconnected-(U1-IO5-Pad29)
- U1 pad 31: unconnected-(U1-IO19-Pad31) -> /OUT_M2_DA
- U1 pad 33: unconnected-(U1-IO21-Pad33) -> /SDA_MPU6050
- U1 pad 36: unconnected-(U1-IO22-Pad36) -> /SCL_MPU6050
- U1 pad 37: unconnected-(U1-IO23-Pad37) -> /IR_FRONTAL
- U1 pad 6: /IR_FRONTAL -> unconnected-(U1-IO34-Pad6)
- U1 pad 7: /IR_IZQ -> /START
- U1 pad 8: unconnected-(U1-IO32-Pad8) -> /IR_DER
- U1 pad 9: unconnected-(U1-IO33-Pad9) -> /M2_IN1
- U2 pad 1: +5V -> +3.3V
- U2 pad 3: /SCL -> /SCL_MPU6050
- U2 pad 4: /SDA -> /SDA_MPU6050
- U2 pad 8: unconnected-(U2-INT-Pad8) -> /INT_MPU6050
- U5 pad 1: unconnected-(U5-nSLEEP-Pad1) -> Net-(U5-nSLEEP)
- U5 pad 10: /BIN2 -> /M1_IN2
- U5 pad 11: unconnected-(U5-VCP-Pad11) -> Net-(U5-VCP)
- U5 pad 12: unconnected-(U5-VM-Pad12) -> +BATT
- U5 pad 14: +BATT -> +3.3V
- U5 pad 15: /AIN2 -> /M2_IN2
- U5 pad 16: /AIN1 -> /M2_IN1
- U5 pad 2: /AOUT1 -> /OUT_B_MOTOR2
- U5 pad 4: /AOUT2 -> /OUT_A_MOTOR2
- U5 pad 5: /BOUT2 -> /OUT_A_MOTOR1
- U5 pad 7: /BOUT1 -> /OUT_B_MOTOR1
- U5 pad 8: unconnected-(U5-nFAULT-Pad8) -> /NFAULT
- U5 pad 9: /BIN1 -> /M1_IN1
- U7 pad 3: +5V -> +BATT
Routing:
- net +3.3V: track 80.0 -> 221.9 mm, vias 0 -> 3
- net +5V: track 249.1 -> 114.7 mm, vias 2 -> 3
- net /START: track 0.00 -> 69.3 mm, vias 0 -> 3
- net /OUT_M1_DB: track 0.00 -> 69.1 mm, vias 0 -> 1
- net +BATT: track 61.9 -> 123.2 mm
- net /OUT_M1_DA: track 0.00 -> 54.6 mm, vias 0 -> 1
- net /OUT_M2_DA: track 0.00 -> 53.4 mm, vias 0 -> 1
- net /D1B: track 46.8 -> 0.00 mm, vias 1 -> 0
- net /D1A: track 45.6 -> 0.00 mm, vias 1 -> 0
- net /M1_IN2: track 0.00 -> 45.6 mm
- net /SCL_MPU6050: track 0.00 -> 44.9 mm, vias 0 -> 1
- net /D2B: track 44.8 -> 0.00 mm, vias 1 -> 0
- net /M1_IN1: track 0.00 -> 43.9 mm
- net /OUT_A_MOTOR2: track 0.00 -> 43.3 mm
- net /start: track 42.0 -> 0.00 mm, vias 1 -> 0
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
Commit message: nueva placa Leandro Flecha verde
Parts:
- removed U4: L7805, EESTN5:SOT223
- added U3: AMS1117-5.0, Package_TO_SOT_SMD:SOT-223-3_TabPin2, F.Cu at (121.3, 84.0)
- C1, C3, C7, C8: footprint EESTN5:C_1206 -> EESTN5:CAP_ELEC_5x11mm
- C10: value C -> 100nF
- J299: footprint EESTN5:SW_SPDT_TH_Vertical -> EESTN5:Pin_Strip_3
- J3: value CP2102 -> Programador; footprint EESTN5:Pin_Header_5 -> EESTN5:pin_strip_4
- J4, J5, J8: footprint Connector_JST:JST_EH_B3B-EH-A_1x03_P2.50mm_Vertical -> EESTN5:Pin_Strip_3
- moved C5 30.8 mm to (116.2, 65.5), turned to -90 degrees
- moved C7 28.9 mm to (112.0, 70.0)
- moved C8 21.1 mm to (125.0, 55.0), turned to 90 degrees
- moved C3 19.6 mm to (113.5, 77.0)
- moved U7 19.6 mm to (122.5, 65.0), turned to 0 degrees
- moved J8 19.3 mm to (166.0, 47.5), turned to 90 degrees
- moved R3 17.8 mm to (144.5, 83.8)
- moved LED_ESP32 16.5 mm to (130.2, 52.0)
- moved R1 16.4 mm to (133.0, 52.0), turned to -90 degrees
- moved U5 15.9 mm to (149.2, 84.0)
- moved C12 15.2 mm to (144.8, 75.6)
- moved C13 15.2 mm to (148.5, 75.6)
- moved C11 15.1 mm to (152.1, 75.6), turned to 90 degrees
- moved C4 14.9 mm to (113.6, 81.7), turned to 180 degrees
- moved C6 14.4 mm to (125.0, 60.0)
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Connections:
- J1 pad 3: +3.3V -> +5V
- J2 pad 3: +3.3V -> +5V
- J3 pad 1: /TX -> /RX
- J3 pad 2: /RX -> /TX
- J3 pad 3: unconnected-(J3-Pin_3-Pad3) -> +5V
- R1 pad 1: +3.3V -> Net-(LED_ESP32-A)
- R1 pad 2: Net-(LED_ESP32-A) -> /EN
- R2 pad 1: +3.3V -> +5V
- U1 pad 10: /M2_IN2 -> /OUT_M2_DA
- U1 pad 11: /M1_IN2 -> /M2_IN1
- U1 pad 12: /M1_IN1 -> /M2_IN2
- U1 pad 30: /OUT_M2_DB -> /M1_IN2
- U1 pad 31: /OUT_M2_DA -> /M1_IN1
- U1 pad 9: /M2_IN1 -> /OUT_M2_DB
Routing:
- net +5V: track 114.7 -> 203.5 mm, vias 3 -> 0
- net +3.3V: track 221.9 -> 152.7 mm, vias 3 -> 0
- net /OUT_M1_DB: track 69.1 -> 0.00 mm, vias 1 -> 0
- net +BATT: track 123.2 -> 60.1 mm, vias 2 -> 0
- net /OUT_M1_DA: track 54.6 -> 0.00 mm, vias 1 -> 0
- net /M1_IN2: track 45.6 -> 0.00 mm
- net /M1_IN1: track 43.9 -> 0.00 mm
- net GND: track 12.2 -> 54.1 mm, vias 1 -> 0
- net /SCL_MPU6050: track 44.9 -> 65.9 mm, vias 1 -> 0
- net /START: track 69.3 -> 89.1 mm, vias 3 -> 1
- net /TX: track 23.3 -> 41.5 mm, vias 1 -> 0
- net /IR_FRONTAL: track 21.4 -> 7.15 mm, vias 1 -> 0
- net /RX: track 24.5 -> 38.3 mm, vias 1 -> 0
- net Net-(U5-VCP): track 12.2 -> 5.01 mm
- net /EN: track 7.17 -> 14.2 mm
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Other:
- board size 100 x 90 mm -> 100 x 99.8 mm
