File: Hardware/Placas Embebidas/Flecha verde/Flecha_Verde_V1.kicad_sch (KiCad schematic)
At the start: 36 parts, among them J2 Jumper, J3 CP2102, J3 Encoder Derecho, J4 Encoder Izquierdo, J5 Distancia_Der, J6 Distancia_Izq, J7 Distancia_Frontal, J8 7.4v, SW1 SW_Push, U1 ESP32-WROOM-32E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

Commit message: Placa terminada
Parts:
- C11, C12, C13, C5, C6, C7, C8: footprint (none) -> EESTN5:C_1206
- J299: renamed from J2; footprint (none) -> EESTN5:SW_SPDT_TH_Vertical
- J3: footprint (none) -> EESTN5:Pin_Header_5
- SW_BOOT1: renamed from SW_BOOT; footprint EESTN5:PUSH_SWITCH_THT -> EESTN5:SW_SPST_EVQPE1
Connections:
- net IR_FRONTAL: now also U1.37 (IO23); no longer U1.26 (IO4)
- net IR_IZQ: now also U1.28 (IO17); no longer U1.37 (IO23)
- net M1_IN1: now also U5.9 (BIN1); no longer U5.16 (AIN1)
- net M1_IN2: now also U5.10 (BIN2); no longer U5.15 (AIN2)
- net M2_IN1: now also U5.16 (AIN1); no longer U5.9 (BIN1)
- net M2_IN2: now also U5.15 (AIN2); no longer U5.10 (BIN2)
- net OUT_A_MOTOR1: now also U5.5 (BOUT2); no longer U5.2 (AOUT1)
- net OUT_A_MOTOR2: now also U5.4 (AOUT2); no longer U5.7 (BOUT1)
- net OUT_B_MOTOR1: now also U5.7 (BOUT1); no longer U5.4 (AOUT2)
- net OUT_B_MOTOR2: now also U5.2 (AOUT1); no longer U5.5 (BOUT2)
- net OUT_M1_DB: now also U1.26 (IO4); no longer U1.28 (IO17)
- net OUT_M2_DA: now also U1.31 (IO19); no longer U1.30 (IO18)
- net OUT_M2_DB: now also U1.30 (IO18); no longer U1.31 (IO19)
- no-connect marks 18 -> 19
Changed lines of the file:
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@@
   (no_connect (at 151.384 66.675))
   (no_connect (at 136.144 89.535))
+  (no_connect (at 133.604 89.535))
   (no_connect (at 143.764 89.535))
   (no_connect (at 113.284 74.295))
@@
     (effects (font (size 3 3) bold) (justify left bottom))
   )
-  (label "OUT_M2_DB" (at 156.464 61.595 0) (fields_autoplaced)
+  (label "OUT_M2_DB" (at 156.464 64.135 0) (fields_autoplaced)
     (effects (font (size 1.27 1.27)) (justify left bottom))
   )
@@
     (effects (font (size 1.27 1.27)) (justify right bottom))
   )
-  (label "OUT_M2_DA" (at 156.464 64.135 0) (fields_autoplaced)
+  (label "OUT_M2_DA" (at 156.464 61.595 0) (fields_autoplaced)
     (effects (font (size 1.27 1.27)) (justify left bottom))
   )
@@
     (effects (font (size 1.27 1.27)) (justify right bottom))
   )
-  (label "M2_IN2" (at 244.856 45.466 0) (fields_autoplaced)
+  (label "M2_IN2" (at 245.364 32.766 0) (fields_autoplaced)
     (effects (font (size 1.27 1.27)) (justify left bottom))
   )
@@
     (effects (font (size 1.27 1.27)) (justify right bottom))
   )
-  (label "OUT_A_MOTOR2" (at 214.884 45.466 180) (fields_autoplaced)
+  (label "OUT_A_MOTOR2" (at 215.392 37.846 180) (fields_autoplaced)
     (effects (font (size 1.27 1.27)) (justify right bottom))
   )
@@
     (effects (font (size 1.27 1.27)) (justify right bottom))
   )
-  (label "OUT_M1_DB" (at 156.464 69.215 0) (fields_autoplaced)
+  (label "OUT_M1_DB" (at 156.464 74.295 0) (fields_autoplaced)
     (effects (font (size 1.27 1.27)) (justify left bottom))
   )
@@
     (effects (font (size 1.27 1.27) italic) (justify right bottom))
   )
-  (label "OUT_B_MOTOR1" (at 215.392 37.846 180) (fields_autoplaced)
+  (label "OUT_B_MOTOR1" (at 214.884 45.466 180) (fields_autoplaced)
     (effects (font (size 1.27 1.27)) (justify right bottom))
   )
@@
     (effects (font (size 1.27 1.27)) (justify right bottom))
   )
-  (label "M1_IN2" (at 245.364 32.766 0) (fields_autoplaced)
+  (label "M1_IN2" (at 244.856 45.466 0) (fields_autoplaced)
     (effects (font (size 1.27 1.27)) (justify left bottom))
   )
@@
     (effects (font (size 1.27 1.27)) (justify right bottom))
   )
-  (label "IR_IZQ" (at 152.019 46.355 0) (fields_autoplaced)
+  (label "IR_IZQ" (at 156.464 69.215 0) (fields_autoplaced)
     (effects (font (size 1.27 1.27)) (justify left bottom))
   )
-  (label "M2_IN1" (at 244.856 48.006 0) (fields_autoplaced)
+  (label "M2_IN1" (at 245.364 30.226 0) (fields_autoplaced)
     (effects (font (size 1.27 1.27)) (justify left bottom))
   )
-  (label "IR_FRONTAL" (at 156.464 74.295 0) (fields_autoplaced)
+  (label "IR_FRONTAL" (at 152.019 46.355 0) (fields_autoplaced)
     (effects (font (size 1.27 1.27)) (justify left bottom))
   )
@@
     (effects (font (size 1.27 1.27)) (justify right bottom))
   )
-  (label "OUT_A_MOTOR1" (at 214.884 32.766 180) (fields_autoplaced)
+  (label "OUT_A_MOTOR1" (at 215.519 40.386 180) (fields_autoplaced)
     (effects (font (size 1.27 1.27)) (justify right bottom))
   )
-  (label "M1_IN1" (at 245.364 30.226 0) (fields_autoplaced)
+  (label "M1_IN1" (at 244.856 48.006 0) (fields_autoplaced)
     (effects (font (size 1.27 1.27)) (justify left bottom))
   )
@@
     (effects (font (size 1.27 1.27)) (justify left bottom))
   )
-  (label "OUT_B_MOTOR2" (at 215.519 40.386 180) (fields_autoplaced)
+  (label "OUT_B_MOTOR2" (at 214.884 32.766 180) (fields_autoplaced)
     (effects (font (size 1.27 1.27)) (justify right bottom))
   )
@@
       (effects (font (size 1.27 1.27)) (justify left))
     )
-    (property "Footprint" "" (at 49.911 145.542 0)
+    (property "Footprint" "EESTN5:Pin_Header_5" (at 49.911 145.542 0)
       (effects (font (size 1.27 1.27)) hide)
     )
@@
   (symbol (lib_id "EESTN5:SW_Push") (at 72.39 185.547 0) (unit 1)
     (in_bom yes) (on_board yes) (dnp no)
-    (property "Reference" "SW_BOOT" (at 70.866 181.102 0)
+    (property "Reference" "SW_BOOT1" (at 70.866 181.102 0)
       (effects (font (size 1.27 1.27)))
     )
@@
       (effects (font (size 1.27 1.27)) hide)
     )
-    (property "Footprint" "EESTN5:PUSH_SWITCH_THT" (at 72.39 180.467 0)
+    (property "Footprint" "EESTN5:SW_SPST_EVQPE1" (at 72.39 180.467 0)
       (effects (font (size 1.27 1.27)) hide)
     )
@@
       (project "Flecha_Verde_V1"
         (path "/b7bd9da0-65fe-4d59-8fc7-564649d3d9ed"
-          (reference "SW_BOOT") (unit 1)
+          (reference "SW_BOOT1") (unit 1)
         )
       )
@@
       (effects (font (size 1.27 1.27)) (justify left))
     )
-    (property "Footprint" "" (at 17.526 31.496 0)
+    (property "Footprint" "EESTN5:C_1206" (at 17.526 31.496 0)
       (effects (font (size 1.27 1.27)) hide)
     )
@@
       (project "Flecha_Verde_V1"
         (path "/b7bd9da0-65fe-4d59-8fc7-564649d3d9ed"
-          (reference "SW_START") (unit 1)
+          (reference "SW_START1") (unit 1)
         )
       )
@@
       (effects (font (size 1.27 1.27)) (justify left))
     )
-    (property "Footprint" "" (at 29.718 31.496 0)
+    (property "Footprint" "EESTN5:C_1206" (at 29.718 31.496 0)
       (effects (font (size 1.27 1.27)) hide)
     )
@@
       (effects (font (size 1.27 1.27)) (justify left))
     )
-    (property "Footprint" "" (at 267.589 36.322 0)
+    (property "Footprint" "EESTN5:C_1206" (at 267.589 36.322 0)
       (effects (font (size 1.27 1.27)) hide)
     )
@@
       (effects (font (size 1.27 1.27)) (justify left))
     )
-    (property "Footprint" "" (at 52.324 32.258 0)
+    (property "Footprint" "EESTN5:C_1206" (at 52.324 32.258 0)
       (effects (font (size 1.27 1.27)) hide)
     )
@@
   (symbol (lib_id "Connector_Generic:Conn_01x03") (at 34.29 190.627 270) (unit 1)
     (in_bom yes) (on_board yes) (dnp no) (fields_autoplaced)
-    (property "Reference" "J2" (at 38.862 189.9833 90)
+    (property "Reference" "J299" (at 39.37 189.992 90)
       (effects (font (size 1.27 1.27)) (justify left))
     )
-    (property "Value" "Jumper" (at 38.862 191.9043 90)
+    (property "Value" "Jumper" (at 39.37 192.532 90)
       (effects (font (size 1.27 1.27)) (justify left))
     )
-    (property "Footprint" "" (at 34.29 190.627 0)
+    (property "Footprint" "EESTN5:SW_SPDT_TH_Vertical" (at 34.29 190.627 0)
       (effects (font (size 1.27 1.27)) hide)
     )
@@
       (project "Flecha_Verde_V1"
         (path "/b7bd9da0-65fe-4d59-8fc7-564649d3d9ed"
-          (reference "J2") (unit 1)
+          (reference "J299") (unit 1)
         )
       )
@@
       (effects (font (size 1.27 1.27)))
     )
-    (property "Footprint" "" (at 257.81 35.306 0)
+    (property "Footprint" "EESTN5:C_1206" (at 257.81 35.306 0)
       (effects (font (size 1.27 1.27)) hide)
     )
@@
       (effects (font (size 1.27 1.27)) (justify left))
     )
-    (property "Footprint" "" (at 59.817 31.877 0)
+    (property "Footprint" "EESTN5:C_1206" (at 59.817 31.877 0)
       (effects (font (size 1.27 1.27)) hide)
     )
@@
       (effects (font (size 1.27 1.27)) (justify left))
     )
-    (property "Footprint" "" (at 262.255 47.244 0)
+    (property "Footprint" "EESTN5:C_1206" (at 262.255 47.244 0)
       (effects (font (size 1.27 1.27)) hide)
     )
@@
   (symbol (lib_id "Connector_Generic:Conn_01x02") (at 15.875 185.547 180) (unit 1)
     (in_bom yes) (on_board yes) (dnp no) (fields_autoplaced)
-    (property "Reference" "J8" (at 15.875 178.7271 0)
+    (property "Reference" "J8" (at 15.875 177.8 0)
       (effects (font (size 1.27 1.27)))
     )
-    (property "Value" "7.4v" (at 15.875 180.6481 0)
+    (property "Value" "7.4v" (at 15.875 180.34 0)
       (effects (font (size 1.27 1.27)))
     )
@@
       (project "Flecha_Verde_V1"
         (path "/b7bd9da0-65fe-4d59-8fc7-564649d3d9ed"
-          (reference "J1") (unit 1)
+          (reference "J199") (unit 1)
         )
       )

Commit message: nueva placa Leandro Flecha verde
Parts:
- removed J3: CP2102, EESTN5:Pin_Header_5, symbol Connector_Generic:Conn_01x05
- removed U1: L7805, EESTN5:SOT223, symbol Regulator_Linear:L7805
- added J3: Programador, EESTN5:pin_strip_4, symbol EESTN5:Conn_01x04
- added U3: AMS1117-5.0, Package_TO_SOT_SMD:SOT-223-3_TabPin2, symbol Regulator_Linear:AMS1117-5.0
- C1, C3, C7, C8: footprint EESTN5:C_1206 -> EESTN5:CAP_ELEC_5x11mm
- C10: value C -> 100nF
- J299: footprint EESTN5:SW_SPDT_TH_Vertical -> EESTN5:Pin_Strip_3
- J5, J6, J7: footprint Connector_JST:JST_EH_B3B-EH-A_1x03_P2.50mm_Vertical -> EESTN5:Pin_Strip_3
Connections:
- net +3.3V: no longer J3.3 (Pin_3), J4.3 (Pin_3), R2.1, R3.1
- net +5V: now also J3.3 (Pin_3), J4.3 (Pin_3), R2.1, J3.3 (Pin_3), U3.2 (VO)
- net +BATT: now also U3.3 (VI)
- net EN: now also R3.2
- net GND: now also J3.4 (Pin_4), U3.1 (GND)
- net M1_IN1: now also U1.31 (IO19); no longer U1.12 (IO27)
- net M1_IN2: now also U1.30 (IO18); no longer U1.11 (IO26)
- net M2_IN1: now also U1.11 (IO26); no longer U1.9 (IO33)
- net M2_IN2: now also U1.12 (IO27); no longer U1.10 (IO25)
- net OUT_M2_DA: now also U1.10 (IO25); no longer U1.31 (IO19)
- net OUT_M2_DB: now also U1.9 (IO33); no longer U1.30 (IO18)
- net RX: now also J3.1 (Pin_1)
- net TX: now also J3.2 (Pin_2)
- net at LED1.1 (A): now also R3.1; no longer R3.2
- no-connect marks 19 -> 18
Other:
- moved on the sheet: R3
