File: Hardware/Placas Embebidas/BoverJr_PCBWAY/_autosave-BoverJr_PCBWAY.kicad_sch (KiCad schematic)
At the start: 46 parts, among them J11 Cable_PAD, J3 Encoder Derecho, J3 Programador, J4 Encoder Izquierdo, J5 Distancia_Der, J6 Cable_PAD, J6 Distancia_Izq, J7 Cable_PAD, J7 Distancia_Frontal, J8 7.4v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

Commit message: estoy verificando por 3d
Parts:
- added G4: LOGO, EESTN5:ezequiel, symbol NOMBRES2:LOGO
- added G5: LOGO, EESTN5:Leandro, symbol NOMBRES:LOGO
- added G6: LOGO, EESTN5:BOVER_NAME, symbol NAME_BOVER:LOGO
Changed lines of the file:
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@@
   (symbol (lib_id "NOMBRES:LOGO") (at 62.9158 100.8888 0) (unit 1)
     (in_bom yes) (on_board yes) (dnp no) (fields_autoplaced)
-    (property "Reference" "#G2" (at 62.9158 99.7872 0)
+    (property "Reference" "G5" (at 62.9158 99.7872 0)
       (effects (font (size 1.27 1.27)) hide)
     )
@@
       (effects (font (size 1.27 1.27)) hide)
     )
-    (property "Footprint" "" (at 62.9158 100.8888 0)
+    (property "Footprint" "EESTN5:Leandro" (at 62.9158 100.8888 0)
       (effects (font (size 1.27 1.27)) hide)
     )
@@
       (project "BoverJr_PCBWAY"
         (path "/b7bd9da0-65fe-4d59-8fc7-564649d3d9ed"
-          (reference "#G2") (unit 1)
+          (reference "G5") (unit 1)
         )
       )
@@
   (symbol (lib_id "NOMBRES2:LOGO") (at 62.9158 95.885 0) (unit 1)
     (in_bom yes) (on_board yes) (dnp no) (fields_autoplaced)
-    (property "Reference" "#G1" (at 62.9158 94.7109 0)
+    (property "Reference" "G4" (at 62.9158 94.7109 0)
       (effects (font (size 1.27 1.27)) hide)
     )
@@
       (effects (font (size 1.27 1.27)) hide)
     )
-    (property "Footprint" "" (at 62.9158 95.885 0)
+    (property "Footprint" "EESTN5:ezequiel" (at 62.9158 95.885 0)
       (effects (font (size 1.27 1.27)) hide)
     )
@@
       (project "BoverJr_PCBWAY"
         (path "/b7bd9da0-65fe-4d59-8fc7-564649d3d9ed"
-          (reference "#G1") (unit 1)
+          (reference "G4") (unit 1)
         )
       )
@@
         )
       )
+    )
+  )
+  (symbol (lib_id "NAME_BOVER:LOGO") (at 62.6364 107.442 0) (unit 1)
+    (in_bom yes) (on_board yes) (dnp no) (fields_autoplaced)
+    (property "Reference" "G6" (at 62.6364 104.7064 0)
+      (effects (font (size 1.27 1.27)) hide)
+    )
+    (property "Value" "LOGO" (at 62.6364 110.1776 0)
+      (effects (font (size 1.27 1.27)) hide)
+    )
+    (property "Footprint" "EESTN5:BOVER_NAME" (at 62.6364 107.442 0)
+      (effects (font (size 1.27 1.27)) hide)
+    )
+    (property "Datasheet" "" (at 62.6364 107.442 0)
+      (effects (font (size 1.27 1.27)) hide)
+    )
+    (instances
+      (project "BoverJr_PCBWAY"
+        (path "/b7bd9da0-65fe-4d59-8fc7-564649d3d9ed"
+          (reference "G6") (unit 1)
+        )
+      )
