File: Hardware/Placas Embebidas/BoverJr_PCBWAY/BoverJr_PCBWAY.kicad_sch (KiCad schematic)
At the start: 46 parts, among them J11 Cable_PAD, J3 Encoder Derecho, J3 Programador, J4 Encoder Izquierdo, J5 Distancia_Der, J6 Cable_PAD, J6 Distancia_Izq, J7 Cable_PAD, J7 Distancia_Frontal, J8 7.4v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

Commit message: soy un boludo
Parts:
- added G4: LOGO, EESTN5:ezequiel, symbol NOMBRES2:LOGO
- added G5: LOGO, EESTN5:Leandro, symbol NOMBRES:LOGO
- added G6: LOGO, EESTN5:BOVER_NAME, symbol NAME_BOVER:LOGO
Changed lines of the file:
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@@
   (symbol (lib_id "NOMBRES:LOGO") (at 62.9158 100.8888 0) (unit 1)
     (in_bom yes) (on_board yes) (dnp no) (fields_autoplaced)
-    (property "Reference" "#G2" (at 62.9158 99.7872 0)
+    (property "Reference" "G5" (at 62.9158 99.7872 0)
       (effects (font (size 1.27 1.27)) hide)
     )
@@
       (effects (font (size 1.27 1.27)) hide)
     )
-    (property "Footprint" "" (at 62.9158 100.8888 0)
+    (property "Footprint" "EESTN5:Leandro" (at 62.9158 100.8888 0)
       (effects (font (size 1.27 1.27)) hide)
     )
@@
       (project "BoverJr_PCBWAY"
         (path "/b7bd9da0-65fe-4d59-8fc7-564649d3d9ed"
-          (reference "#G2") (unit 1)
+          (reference "G5") (unit 1)
         )
       )
@@
   (symbol (lib_id "NOMBRES2:LOGO") (at 62.9158 95.885 0) (unit 1)
     (in_bom yes) (on_board yes) (dnp no) (fields_autoplaced)
-    (property "Reference" "#G1" (at 62.9158 94.7109 0)
+    (property "Reference" "G4" (at 62.9158 94.7109 0)
       (effects (font (size 1.27 1.27)) hide)
     )
@@
       (effects (font (size 1.27 1.27)) hide)
     )
-    (property "Footprint" "" (at 62.9158 95.885 0)
+    (property "Footprint" "EESTN5:ezequiel" (at 62.9158 95.885 0)
       (effects (font (size 1.27 1.27)) hide)
     )
@@
       (project "BoverJr_PCBWAY"
         (path "/b7bd9da0-65fe-4d59-8fc7-564649d3d9ed"
-          (reference "#G1") (unit 1)
+          (reference "G4") (unit 1)
         )
       )
@@
         )
       )
+    )
+  )
+  (symbol (lib_id "NAME_BOVER:LOGO") (at 61.8744 111.4044 0) (unit 1)
+    (in_bom yes) (on_board yes) (dnp no) (fields_autoplaced)
+    (property "Reference" "G6" (at 61.8744 108.6688 0)
+      (effects (font (size 1.27 1.27)) hide)
+    )
+    (property "Value" "LOGO" (at 61.8744 114.14 0)
+      (effects (font (size 1.27 1.27)) hide)
+    )
+    (property "Footprint" "EESTN5:BOVER_NAME" (at 61.8744 111.4044 0)
+      (effects (font (size 1.27 1.27)) hide)
+    )
+    (property "Datasheet" "" (at 61.8744 111.4044 0)
+      (effects (font (size 1.27 1.27)) hide)
+    )
+    (instances
+      (project "BoverJr_PCBWAY"
+        (path "/b7bd9da0-65fe-4d59-8fc7-564649d3d9ed"
+          (reference "G6") (unit 1)
+        )
+      )

Commit message: Para mi esat lista , verificada por 3D y ezequiel, faltaria saber que dice bustos
Parts:
- removed G4: LOGO, EESTN5:ezequiel, symbol NOMBRES2:LOGO
- removed G5: LOGO, EESTN5:Leandro, symbol NOMBRES:LOGO
- added G8: LOGO_ROTULO, EESTN5:LOGO_EESTN5_F.Cu, symbol EESTN5:LOGO_ROTULO
- J3: footprint EESTN5:pin_strip_4 -> Connector_PinSocket_2.54mm:PinSocket_1x04_P2.54mm_Vertical
- J5, J6, J7: footprint EESTN5:Pin_Strip_3 -> Connector_JST:JST_XH_B3B-XH-AM_1x03_P2.50mm_Vertical
- R2, R3, R7, R8: footprint EESTN5:R_1206 -> EESTN5:R_0805
Changed lines of the file:
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@@
       (effects (font (size 1.27 1.27)) (justify left))
     )
-    (property "Footprint" "EESTN5:Pin_Strip_3" (at 264.033 100.076 0)
+    (property "Footprint" "Connector_JST:JST_XH_B3B-XH-AM_1x03_P2.50mm_Vertical" (at 264.033 100.076 0)
       (effects (font (size 1.27 1.27)) hide)
     )
@@
     )
   )
-  (symbol (lib_id "NOMBRES:LOGO") (at 62.9158 100.8888 0) (unit 1)
-    (in_bom yes) (on_board yes) (dnp no) (fields_autoplaced)
-    (property "Reference" "G5" (at 62.9158 99.7872 0)
-      (effects (font (size 1.27 1.27)) hide)
-    )
-    (property "Value" "LOGO" (at 62.9158 101.9904 0)
-      (effects (font (size 1.27 1.27)) hide)
-    )
-    (property "Footprint" "EESTN5:Leandro" (at 62.9158 100.8888 0)
-      (effects (font (size 1.27 1.27)) hide)
-    )
-    (property "Datasheet" "" (at 62.9158 100.8888 0)
-      (effects (font (size 1.27 1.27)) hide)
-    )
-    (instances
-      (project "BoverJr_PCBWAY"
-        (path "/b7bd9da0-65fe-4d59-8fc7-564649d3d9ed"
-          (reference "G5") (unit 1)
+  (symbol (lib_id "EESTN5:LOGO_ROTULO") (at 61.5442 95.758 0) (unit 1)
+    (in_bom yes) (on_board yes) (dnp no) (fields_autoplaced)
+    (property "Reference" "G8" (at 61.5442 101.3968 0)
+      (effects (font (size 1.524 1.524)) hide)
+    )
+    (property "Value" "LOGO_ROTULO" (at 61.5442 90.1192 0)
+      (effects (font (size 1.524 1.524)) hide)
+    )
+    (property "Footprint" "EESTN5:LOGO_EESTN5_F.Cu" (at 61.5442 95.758 0)
+      (effects (font (size 1.524 1.524)) hide)
+    )
+    (property "Datasheet" "" (at 61.5442 95.758 0)
+      (effects (font (size 1.524 1.524)) hide)
+    )
+    (instances
+      (project "BoverJr_PCBWAY"
+        (path "/b7bd9da0-65fe-4d59-8fc7-564649d3d9ed"
+          (reference "G8") (unit 1)
         )
       )
@@
     )
   )
-  (symbol (lib_id "NOMBRES2:LOGO") (at 62.9158 95.885 0) (unit 1)
-    (in_bom yes) (on_board yes) (dnp no) (fields_autoplaced)
-    (property "Reference" "G4" (at 62.9158 94.7109 0)
-      (effects (font (size 1.27 1.27)) hide)
-    )
-    (property "Value" "LOGO" (at 62.9158 97.0591 0)
-      (effects (font (size 1.27 1.27)) hide)
-    )
-    (property "Footprint" "EESTN5:ezequiel" (at 62.9158 95.885 0)
-      (effects (font (size 1.27 1.27)) hide)
-    )
-    (property "Datasheet" "" (at 62.9158 95.885 0)
-      (effects (font (size 1.27 1.27)) hide)
-    )
-    (instances
-      (project "BoverJr_PCBWAY"
-        (path "/b7bd9da0-65fe-4d59-8fc7-564649d3d9ed"
-          (reference "G4") (unit 1)
-        )
-      )
-    )
-  )
   (symbol (lib_id "EESTN5:C") (at 146.05 184.785 90) (unit 1)
     (in_bom yes) (on_board yes) (dnp no)
@@
       (effects (font (size 1.27 1.27)))
     )
-    (property "Footprint" "EESTN5:R_1206" (at 83.82 180.34 0)
+    (property "Footprint" "EESTN5:R_0805" (at 83.82 180.34 0)
       (effects (font (size 1.524 1.524)) hide)
     )
@@
       (effects (font (size 1.27 1.27)) (justify right))
     )
-    (property "Footprint" "EESTN5:R_1206" (at 72.136 23.622 90)
+    (property "Footprint" "EESTN5:R_0805" (at 72.136 23.622 90)
       (effects (font (size 1.27 1.27)) hide)
     )
@@
       (effects (font (size 1.27 1.27)) (justify left))
     )
-    (property "Footprint" "EESTN5:pin_strip_4" (at 156.4386 146.3294 0)
+    (property "Footprint" "Connector_PinSocket_2.54mm:PinSocket_1x04_P2.54mm_Vertical" (at 156.4386 146.3294 0)
       (effects (font (size 1.27 1.27)) hide)
     )
@@
       (effects (font (size 1.27 1.27)) (justify left))
     )
-    (property "Footprint" "EESTN5:R_1206" (at 195.834 26.416 90)
+    (property "Footprint" "EESTN5:R_0805" (at 195.834 26.416 90)
       (effects (font (size 1.27 1.27)) hide)
     )
@@
       (effects (font (size 1.27 1.27)))
     )
-    (property "Footprint" "EESTN5:R_1206" (at 126.9492 184.9374 0)
+    (property "Footprint" "EESTN5:R_0805" (at 126.9492 184.9374 0)
       (effects (font (size 1.524 1.524)) hide)
     )
@@
       (effects (font (size 1.27 1.27)))
     )
-    (property "Footprint" "EESTN5:R_1206" (at 159.385 179.07 0)
+    (property "Footprint" "EESTN5:R_0805" (at 159.385 179.07 0)
       (effects (font (size 1.524 1.524)) hide)
     )
@@
       (effects (font (size 1.27 1.27)) (justify left))
     )
-    (property "Footprint" "EESTN5:Pin_Strip_3" (at 264.033 73.406 0)
+    (property "Footprint" "Connector_JST:JST_XH_B3B-XH-AM_1x03_P2.50mm_Vertical" (at 264.033 73.406 0)
       (effects (font (size 1.27 1.27)) hide)
     )
@@
       (effects (font (size 1.27 1.27)) (justify left))
     )
-    (property "Footprint" "EESTN5:Pin_Strip_3" (at 264.033 87.63 0)
-      (effects (font (size 1.27 1.27)) hide)
-    )
+    (property "Footprint" "Connector_JST:JST_XH_B3B-XH-AM_1x03_P2.50mm_Vertical" (at 264.033 87.63 0)
+      (effects (font (size 1.27 1.27)) hide)
+    )

Commit message: cosas por mejorar
Parts:
- removed G8: LOGO_ROTULO, EESTN5:LOGO_EESTN5_F.Cu, symbol EESTN5:LOGO_ROTULO
- added G10: LOGO, EESTN5:Leandro, symbol NOMBRES:LOGO
- added G11: LOGO, EESTN5:ezequiel, symbol NOMBRES2:LOGO
Changed lines of the file:
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@@
-    )
-  )
-  (symbol (lib_id "EESTN5:LOGO_ROTULO") (at 61.5442 95.758 0) (unit 1)
-    (in_bom yes) (on_board yes) (dnp no) (fields_autoplaced)
-    (property "Reference" "G8" (at 61.5442 101.3968 0)
-      (effects (font (size 1.524 1.524)) hide)
-    )
-    (property "Value" "LOGO_ROTULO" (at 61.5442 90.1192 0)
-      (effects (font (size 1.524 1.524)) hide)
-    )
-    (property "Footprint" "EESTN5:LOGO_EESTN5_F.Cu" (at 61.5442 95.758 0)
-      (effects (font (size 1.524 1.524)) hide)
-    )
-    (property "Datasheet" "" (at 61.5442 95.758 0)
-      (effects (font (size 1.524 1.524)) hide)
-    )
-    (instances
-      (project "BoverJr_PCBWAY"
-        (path "/b7bd9da0-65fe-4d59-8fc7-564649d3d9ed"
-          (reference "G8") (unit 1)
-        )
-      )
     )
   )
@@
     )
   )
+  (symbol (lib_id "NOMBRES:LOGO") (at 62.4586 92.5576 0) (unit 1)
+    (in_bom yes) (on_board yes) (dnp no) (fields_autoplaced)
+    (property "Reference" "G10" (at 62.4586 91.456 0)
+      (effects (font (size 1.27 1.27)) hide)
+    )
+    (property "Value" "LOGO" (at 62.4586 93.6592 0)
+      (effects (font (size 1.27 1.27)) hide)
+    )
+    (property "Footprint" "EESTN5:Leandro" (at 62.4586 92.5576 0)
+      (effects (font (size 1.27 1.27)) hide)
+    )
+    (property "Datasheet" "" (at 62.4586 92.5576 0)
+      (effects (font (size 1.27 1.27)) hide)
+    )
+    (instances
+      (project "BoverJr_PCBWAY"
+        (path "/b7bd9da0-65fe-4d59-8fc7-564649d3d9ed"
+          (reference "G10") (unit 1)
+        )
+      )
+    )
+  )
   (symbol (lib_id "power:GND") (at 98.3234 186.7662 0) (unit 1)
     (in_bom yes) (on_board yes) (dnp no)
@@
         )
       )
+    )
+  )
+  (symbol (lib_id "NOMBRES2:LOGO") (at 62.4586 99.4664 0) (unit 1)
+    (in_bom yes) (on_board yes) (dnp no) (fields_autoplaced)
+    (property "Reference" "G11" (at 62.4586 98.2923 0)
+      (effects (font (size 1.27 1.27)) hide)
+    )
+    (property "Value" "LOGO" (at 62.4586 100.6405 0)
+      (effects (font (size 1.27 1.27)) hide)
+    )
+    (property "Footprint" "EESTN5:ezequiel" (at 62.4586 99.4664 0)
+      (effects (font (size 1.27 1.27)) hide)
+    )
+    (property "Datasheet" "" (at 62.4586 99.4664 0)
+      (effects (font (size 1.27 1.27)) hide)
+    )
+    (instances
+      (project "BoverJr_PCBWAY"
+        (path "/b7bd9da0-65fe-4d59-8fc7-564649d3d9ed"
+          (reference "G11") (unit 1)
+        )
+      )

Commit message: para mi ya esta listimisima, cambie sw y agregue jst , verifique serigrafia y 3d
Parts:
- SW1: footprint EESTN5:SW_SPDT_TH_100Mils_VERTICAL -> EESTN5:SW_MINI-SPDT-SW
Changed lines of the file:
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@@
       (effects (font (size 1.27 1.27)) hide)
     )
-    (property "Footprint" "EESTN5:SW_SPDT_TH_100Mils_VERTICAL" (at 35.56 184.15 0)
+    (property "Footprint" "EESTN5:SW_MINI-SPDT-SW" (at 35.56 184.15 0)
       (effects (font (size 1.27 1.27)) hide)
     )
