File: Hardware/Placas Embebidas/BoverJr_PCBWAY/BoverJr_PCBWAY.kicad_sch (KiCad schematic)
At the start: 49 parts, among them J11 Cable_PAD, J3 Encoder Derecho, J3 Programador, J4 Encoder Izquierdo, J5 Distancia_Der, J6 Cable_PAD, J6 Distancia_Izq, J7 Cable_PAD, J7 Distancia_Frontal, J8 7.4v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

Commit message: Placa lista, felicidades
Parts:
- added G14: LOGO, EESTN5:logo_pcbway, symbol pcbway_logo:LOGO
Changed lines of the file:
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@@
+    )
+  )
+  (symbol (lib_id "pcbway_logo:LOGO") (at 60.4774 121.3104 0) (unit 1)
+    (in_bom yes) (on_board yes) (dnp no) (fields_autoplaced)
+    (property "Reference" "G14" (at 60.4774 114.875 0)
+      (effects (font (size 1.27 1.27)) hide)
+    )
+    (property "Value" "LOGO" (at 60.4774 127.7458 0)
+      (effects (font (size 1.27 1.27)) hide)
+    )
+    (property "Footprint" "EESTN5:logo_pcbway" (at 60.4774 121.3104 0)
+      (effects (font (size 1.27 1.27)) hide)
+    )
+    (property "Datasheet" "" (at 60.4774 121.3104 0)
+      (effects (font (size 1.27 1.27)) hide)
+    )
+    (instances
+      (project "BoverJr_PCBWAY"
+        (path "/b7bd9da0-65fe-4d59-8fc7-564649d3d9ed"
+          (reference "G14") (unit 1)
+        )
+      )
     )
   )
