File: Hardware/BoverJR/PCBWAY/Modulo_MPU-9150/PCB-MPU-9150/PCB-MPU-9150.kicad_sch (KiCad schematic)
At the start: 15 parts, among them P1 CONN_01X08, U1 MPU-9150, U2 AP2112K-3.3

Commit message: modifique sch un poco
Other:
- company: (none) -> Bover GROUP
- moved on the sheet: C1, C2, C3, C4, C5, C6, C7, JP1, LED1, P1, R1, R2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
