File: Hardware/BoverJR/PCBWAY/Wakanda_MultiRobot/Wakanda_MultiRobot/Wakanda_MultiRobot.kicad_sch (KiCad schematic)
At the start: 21 parts, among them J3 TATAMI Frontal Derecho, J4 TATAMI Frontal Izquierdo, J6 Programador, P1 Mounting_Hole, P2 Mounting_Hole, P3 Mounting_Hole, P4 Mounting_Hole, SW1 START, SW2 SW_Push, SW3 SW_Push

Commit message: agrego avances
Parts:
- removed C10, C12, C5, C7: 10uF, EESTN5:CAP_TAN_A, symbol Device:C_Polarized
- removed C11, C13: 100nF, EESTN5:C_1206, symbol EESTN5:C
- added C9: 100nF, EESTN5:C_1206, symbol Device:C_Small
- added J1: TB_1X3, symbol EESTN5:TB_1X3
- added U1: ESP32-WROOM-32E, EESTN5:ESP32-WROOM-32E, symbol Librerias:ESP32-WROOM-32E
- added U4: AP2112K-3.3, Package_TO_SOT_SMD:SOT-23-5, symbol Regulator_Linear:AP2112K-3.3
- C6, C8: value 100nF -> 1uF
Connections:
- net Vin is gone; now on net +5V: C6.1
- net +3V3: now also C9.1, U1.3V3, U4.5 (VOUT)
- net +5V: now also J1.3, U4.1 (VIN), U4.3 (EN)
- net EN: now also U1.9 (EN)
- net GND: now also C9.2, J1.2, U1.GND, U4.2 (GND)
- net IO0: now also U1.23 (IO0)
- net M_DER_A: now also U1.16 (IO27)
- net M_DER_B: now also U1.15 (IO26)
- net M_IZQ_A: now also U1.25 (IO16)
- net M_IZQ_B: now also U1.27 (IO17)
- net RXD: now also U1.40 (RXD0)
- net SCL: now also U1.39 (IO22)
- net SDA: now also U1.42 (IO21)
- net SH-DER: now also U1.38 (IO19)
- net SH-IZQ: now also U1.35 (IO18)
- net START: now also U1.11 (IO35)
- net TATAMI_FD: now also U1.13 (IO33)
- net TATAMI_FI: now also U1.12 (IO32)
- net TXD: now also U1.41 (TXD0)
- net WS2812: now also U1.14 (IO25)
- new net +BATT: J1.1
Other:
- moved on the sheet: C8

Commit message: agrego cambios en el sch
Parts:
- added J11: Conn_01x04, symbol EESTN5:Conn_01x04
- added J2: Sensor Distancia 1, symbol EESTN5:Conn_01X03
- added J6, J7, J8: Conn_01X03, symbol EESTN5:Conn_01X03
Connections:
- net +5V: now also J11.3 (Pin_3), J2.1 (P1), J6.1 (P1), J7.1 (P1), J8.1 (P1)
- net GND: now also J11.4 (Pin_4), J2.2 (P2), J6.2 (P2), J7.2 (P2), J8.2 (P2)
- net SCL: now also J11.2 (Pin_2)
- net SDA: now also J11.1 (Pin_1)
- net START: now also U1.10 (IO34); no longer U1.11 (IO35)
- net TATAMI_FD: now also U1.12 (IO32); no longer U1.13 (IO33)
- net TATAMI_FI: now also U1.11 (IO35); no longer U1.12 (IO32)
- net SH-DER renamed SENSOR3
- net SENSOR3: now also J7.3 (P3)
- net SH-IZQ renamed SENSOR4
- net SENSOR4: now also J8.3 (P3)
- net WS2812 renamed SENSOR2
- net SENSOR2: now also J6.3 (P3)
- new net SENSOR1: J2.3 (P3), U1.13 (IO33)
Other:
- note added: "Alimentacion"
- note added: "SALIDAS I2C"
- moved on the sheet: C6, C8, C9, J1, J3, J4, R6, SW1, SW2, SW3, U4

Commit message: ordene PCB
Parts:
- C6, C8, C9: footprint EESTN5:C_1206 -> EESTN5:C_0805
- J1: value TB_1X3 -> Alimentacion; footprint (none) -> EESTN5:BORNERA3_AZUL
- J10: renamed from J11; value Conn_01x04 -> I2C; footprint (none) -> EESTN5:pin_strip_4
- J3: renamed from J2; footprint (none) -> EESTN5:Pin_Header_3
- J4: renamed from J6; footprint (none) -> EESTN5:Pin_Header_3
- J5: renamed from J7; footprint (none) -> EESTN5:Pin_Header_3
- J6: renamed from J8; footprint (none) -> EESTN5:Pin_Header_3
- J6: footprint EESTN5:HEADER-4H -> EESTN5:pin_strip_4
- R6: footprint EESTN5:R_1206 -> EESTN5:R_0805
Other:
- note removed: "SALIDAS I2C"

Commit message: casi termino PCB
Connections:
- net +3V3: no longer SW1.2 (P2)
- net +5V: now also SW1.2 (P2)
- net M_DER_A: now also U1.27 (IO17); no longer U1.16 (IO27)
- net M_DER_B: now also U1.25 (IO16); no longer U1.15 (IO26)
- net M_IZQ_A: now also U1.16 (IO27); no longer U1.25 (IO16)
- net M_IZQ_B: now also U1.15 (IO26); no longer U1.27 (IO17)
- net START: now also U1.11 (IO35); no longer U1.10 (IO34)
- net TATAMI_FD: now also U1.36 (IO23); no longer U1.12 (IO32)
- net TATAMI_FI: now also U1.12 (IO32); no longer U1.11 (IO35)
- net +BATT renamed Vin
Changed lines of the file:
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@@
     (stroke (width 0) (type default))
   )
-  (wire (pts (xy 262.255 30.734) (xy 262.255 28.194))
+  (wire (pts (xy 267.208 30.734) (xy 267.208 28.194))
     (stroke (width 0) (type default))
   )
@@
     (stroke (width 0) (type default))
   )
+  (wire (pts (xy 216.535 45.974) (xy 219.075 45.974))
+    (stroke (width 0) (type default))
+  )
   (wire (pts (xy 101.854 110.363) (xy 113.792 110.363))
     (stroke (width 0) (type default))
@@
     (stroke (width 0) (type default))
   )
-  (wire (pts (xy 63.754 50.419) (xy 74.93 50.419))
+  (wire (pts (xy 254.635 30.734) (xy 252.095 30.734))
     (stroke (width 0) (type default))
   )
-  (wire (pts (xy 135.255 117.856) (xy 135.255 114.173))
+  (wire (pts (xy 63.754 50.419) (xy 74.93 50.419))
     (stroke (width 0) (type default))
   )
-  (wire (pts (xy 216.535 40.894) (xy 219.075 40.894))
+  (wire (pts (xy 135.255 117.856) (xy 135.255 114.173))
     (stroke (width 0) (type default))
   )
@@
     (stroke (width 0) (type default))
   )
+  (wire (pts (xy 216.535 43.434) (xy 219.075 43.434))
+    (stroke (width 0) (type default))
+  )
   (wire (pts (xy 249.047 82.677) (xy 261.62 82.677))
     (stroke (width 0) (type default))
@@
     (stroke (width 0) (type default))
   )
-  (wire (pts (xy 216.535 43.434) (xy 219.075 43.434))
-    (stroke (width 0) (type default))
-  )
   (wire (pts (xy 187.071 59.944) (xy 187.071 57.912))
     (stroke (width 0) (type default))
@@
     (stroke (width 0) (type default))
   )
-  (wire (pts (xy 216.535 45.974) (xy 219.075 45.974))
+  (wire (pts (xy 267.208 28.194) (xy 262.255 28.194))
     (stroke (width 0) (type default))
   )
@@
     (effects (font (size 1.524 1.524) (thickness 0.3048) bold) (justify right bottom))
   )
+  (label "M_DER_B" (at 254.635 56.134 0) (fields_autoplaced)
+    (effects (font (size 1.524 1.524)) (justify left bottom))
+  )
+  (label "TATAMI_FD" (at 254.635 30.734 0) (fields_autoplaced)
+    (effects (font (size 1.524 1.524)) (justify left bottom))
+  )
   (label "SCL" (at 26.162 170.688 180) (fields_autoplaced)
     (effects (font (size 1.27 1.27)) (justify right bottom))
   )
+  (label "M_IZQ_A" (at 216.535 56.134 180) (fields_autoplaced)
+    (effects (font (size 1.524 1.524)) (justify right bottom))
+  )
   (label "SCL" (at 254.635 33.274 0) (fields_autoplaced)
     (effects (font (size 1.27 1.27)) (justify left bottom))
@@
     (effects (font (size 1.27 1.27)) (justify left bottom))
   )
-  (label "START" (at 216.535 40.894 180) (fields_autoplaced)
-    (effects (font (size 1.524 1.524)) (justify right bottom))
-  )
-  (label "TATAMI_FD" (at 216.535 45.974 180) (fields_autoplaced)
-    (effects (font (size 1.524 1.524)) (justify right bottom))
-  )
   (label "GND" (at 141.986 115.316 180) (fields_autoplaced)
     (effects (font (size 1.524 1.524)) (justify right bottom))
@@
     (effects (font (size 1.27 1.27)) (justify left bottom))
   )
-  (label "M_IZQ_A" (at 254.635 56.134 0) (fields_autoplaced)
-    (effects (font (size 1.524 1.524)) (justify left bottom))
-  )
   (label "TXD" (at 256.54 80.137 180) (fields_autoplaced)
     (effects (font (size 1.27 1.27)) (justify right bottom))
   )
-  (label "M_DER_B" (at 216.535 53.594 180) (fields_autoplaced)
-    (effects (font (size 1.524 1.524)) (justify right bottom))
-  )
   (label "SENSOR2" (at 75.438 115.443 180) (fields_autoplaced)
     (effects (font (size 1.27 1.27)) (justify right bottom))
@@
     (effects (font (size 1.524 1.524)) (justify right bottom))
   )
+  (label "M_DER_A" (at 254.635 53.594 0) (fields_autoplaced)
+    (effects (font (size 1.524 1.524)) (justify left bottom))
+  )
   (label "TATAMI_FI" (at 141.986 120.396 180) (fields_autoplaced)
     (effects (font (size 1.524 1.524)) (justify right bottom))
@@
     (effects (font (size 1.27 1.27)) (justify right bottom))
   )
+  (label "START" (at 216.535 43.434 180) (fields_autoplaced)
+    (effects (font (size 1.524 1.524)) (justify right bottom))
+  )
   (label "SDA" (at 26.035 168.148 180) (fields_autoplaced)
     (effects (font (size 1.27 1.27)) (justify right bottom))
@@
     (effects (font (size 1.524 1.524)) (justify right bottom))
   )
-  (label "TATAMI_FI" (at 216.535 43.434 180) (fields_autoplaced)
-    (effects (font (size 1.524 1.524)) (justify right bottom))
-  )
-  (label "M_DER_A" (at 216.535 56.134 180) (fields_autoplaced)
-    (effects (font (size 1.524 1.524)) (justify right bottom))
-  )
   (label "IO0" (at 254.635 61.214 0) (fields_autoplaced)
     (effects (font (size 1.27 1.27)) (justify left bottom))
@@
     (effects (font (size 1.524 1.524)) (justify left bottom))
   )
-  (label "M_IZQ_B" (at 254.635 53.594 0) (fields_autoplaced)
-    (effects (font (size 1.524 1.524)) (justify left bottom))
-  )
   (label "SDA" (at 254.635 40.894 0) (fields_autoplaced)
     (effects (font (size 1.27 1.27)) (justify left bottom))
   )
+  (label "M_IZQ_B" (at 216.535 53.594 180) (fields_autoplaced)
+    (effects (font (size 1.524 1.524)) (justify right bottom))
+  )
   (label "SENSOR4" (at 111.633 115.443 180) (fields_autoplaced)
     (effects (font (size 1.27 1.27)) (justify right bottom))
   )
+  (label "TATAMI_FI" (at 216.535 45.974 180) (fields_autoplaced)
+    (effects (font (size 1.524 1.524)) (justify right bottom))
+  )
+  (global_label "Vin" (shape input) (at 30.861 33.02 0) (fields_autoplaced)
+    (effects (font (size 1.27 1.27)) (justify left))
+    (property "Intersheetrefs" "${INTERSHEET_REFS}" (at 36.6092 33.02 0)
+      (effects (font (size 1.27 1.27)) (justify left) hide)
+    )
+  )
   (symbol (lib_id "EESTN5:SW_Push") (at 187.071 52.832 90) (unit 1)
     (in_bom yes) (on_board yes) (dnp no) (fields_autoplaced)
@@
     )
   )
+  (symbol (lib_id "power:+5V") (at 190.246 99.06 0) (unit 1)
+    (in_bom yes) (on_board yes) (dnp no)
+    (property "Reference" "#PWR04" (at 190.246 102.87 0)
+      (effects (font (size 1.27 1.27)) hide)
+    )
+    (property "Value" "+5V" (at 190.246 95.504 0)
+      (effects (font (size 1.27 1.27)))
+    )
+    (property "Footprint" "" (at 190.246 99.06 0)
+      (effects (font (size 1.27 1.27)) hide)
+    )
+    (property "Datasheet" "" (at 190.246 99.06 0)
+      (effects (font (size 1.27 1.27)) hide)
+    )
+    (pin "1")
+    (instances
+      (project "wakanda-board"
+        (path "/19267798-4e4c-4aeb-bec3-b7452995418d"
+          (reference "#PWR04") (unit 1)
+        )
+      )
+      (project "2022-XDecito"
+        (path "/5528bcad-2950-4673-90eb-c37e6952c475"
+          (reference "#PWR05") (unit 1)
+        )
+      )
+      (project "Wakanda_MultiRobot"
+        (path "/7706e104-9d42-4651-8ea1-0974927a2230"
+          (reference "#PWR035") (unit 1)
+        )
+      )
+    )
+  )
   (symbol (lib_id "power:+3V3") (at 187.071 32.385 0) (unit 1)
     (in_bom yes) (on_board yes) (dnp no) (fields_autoplaced)
@@
     )
   )
-  (symbol (lib_id "power:GND") (at 262.255 30.734 0) (unit 1)
+  (symbol (lib_id "power:GND") (at 267.208 30.734 0) (unit 1)
     (in_bom yes) (on_board yes) (dnp no) (fields_autoplaced)
-    (property "Reference" "#PWR020" (at 262.255 37.084 0)
+    (property "Reference" "#PWR020" (at 267.208 37.084 0)
       (effects (font (size 1.27 1.27)) hide)
     )
-    (property "Value" "GND" (at 262.255 36.1442 0)
+    (property "Value" "GND" (at 267.208 36.1442 0)
       (effects (font (size 1.27 1.27)))
     )
-    (property "Footprint" "" (at 262.255 30.734 0)
+    (property "Footprint" "" (at 267.208 30.734 0)
       (effects (font (size 1.27 1.27)) hide)
     )
-    (property "Datasheet" "" (at 262.255 30.734 0)
+    (property "Datasheet" "" (at 267.208 30.734 0)
       (effects (font (size 1.27 1.27)) hide)
     )
@@
     )
   )
-  (symbol (lib_id "power:+BATT") (at 30.861 33.02 0) (unit 1)
-    (in_bom yes) (on_board yes) (dnp no) (fields_autoplaced)
-    (property "Reference" "#PWR08" (at 30.861 36.83 0)
-      (effects (font (size 1.27 1.27)) hide)
-    )
-    (property "Value" "+BATT" (at 30.861 29.591 0)
-      (effects (font (size 1.27 1.27)))
-    )
-    (property "Footprint" "" (at 30.861 33.02 0)
-      (effects (font (size 1.27 1.27)) hide)
-    )
-    (property "Datasheet" "" (at 30.861 33.02 0)
-      (effects (font (size 1.27 1.27)) hide)
-    )
-    (pin "1")
-    (instances
-      (project "Wakanda_MultiRobot"
-        (path "/7706e104-9d42-4651-8ea1-0974927a2230"
-          (reference "#PWR08") (unit 1)
-        )
-      )
-    )
-  )
   (symbol (lib_id "power:GND") (at 208.915 30.734 0) (unit 1)
     (in_bom yes) (on_board yes) (dnp no) (fields_autoplaced)
@@
         )
       )
-    )
-  )
-  (symbol (lib_id "power:+3V3") (at 190.246 99.06 0) (unit 1)
-    (in_bom yes) (on_board yes) (dnp no) (fields_autoplaced)
-    (property "Reference" "#PWR027" (at 190.246 102.87 0)
-      (effects (font (size 1.27 1.27)) hide)
-    )
-    (property "Value" "+3V3" (at 190.246 95.25 0)
-      (effects (font (size 1.27 1.27)))
-    )
-    (property "Footprint" "" (at 190.246 99.06 0)
-      (effects (font (size 1.27 1.27)) hide)
-    )
-    (property "Datasheet" "" (at 190.246 99.06 0)
-      (effects (font (size 1.27 1.27)) hide)
-    )
-    (pin "1")
-    (instances
-      (project "wakanda-board"
-        (path "/19267798-4e4c-4aeb-bec3-b7452995418d"
-          (reference "#PWR027") (unit 1)
-        )
-      )
-      (project "Wakanda_MultiRobot"
-        (path "/7706e104-9d42-4651-8ea1-0974927a2230"
-          (reference "#PWR02") (unit 1)
-        )
-      )

Commit message: placa casi terminada falta 3d y estetica
Other:
- note added: "PROGRAMACION"
- note added: "SALIDA I2C"
- moved on the sheet: C9, J10, J3, J4, J5, J6, R6, SW1, SW2, SW3

Commit message: verifique por 3d
Parts:
- J3, J4: footprint EESTN5:Pin_Strip_3 -> EESTN5:Pin_Header_3
- renumbered J4 to J2
Changed lines of the file:
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@@
   (symbol (lib_id "EESTN5:Conn_01X03") (at 82.677 112.903 0) (unit 1)
     (in_bom yes) (on_board yes) (dnp no) (fields_autoplaced)
-    (property "Reference" "J4" (at 85.09 113.538 0)
+    (property "Reference" "J2" (at 85.09 113.538 0)
       (effects (font (size 1.27 1.27)) (justify left))
     )
@@
       (project "Wakanda_MultiRobot"
         (path "/7706e104-9d42-4651-8ea1-0974927a2230"
-          (reference "J4") (unit 1)
+          (reference "J2") (unit 1)
         )
       )
@@
       (effects (font (size 1.27 1.27)))
     )
-    (property "Footprint" "EESTN5:Pin_Strip_3" (at 145.034 117.348 0)
+    (property "Footprint" "EESTN5:Pin_Header_3" (at 145.034 117.348 0)
       (effects (font (size 1.27 1.27)) hide)
     )
@@
       (effects (font (size 1.27 1.27)))
     )
-    (property "Footprint" "EESTN5:Pin_Strip_3" (at 145.034 94.488 0)
-      (effects (font (size 1.27 1.27)) hide)
-    )
+    (property "Footprint" "EESTN5:Pin_Header_3" (at 145.034 94.488 0)
+      (effects (font (size 1.27 1.27)) hide)
+    )

Commit message: recomendacion de bustos
Parts:
- added J14: RANDOM, EESTN5:pin_strip_4, symbol EESTN5:Conn_01x04
- added J4: Conn_01X03, EESTN5:Pin_Header_3, symbol EESTN5:Conn_01X03
Connections:
- net +5V: now also J14.1 (Pin_1), J4.2 (P2)
- net GND: now also J14.4 (Pin_4), J4.1 (P1)
- net SENSOR5: now reaches U1.10 (IO34)
- net SENSOR5: now also J4.3 (P3)
- net GPIO4: now reaches U1.24 (IO4)
- net GPIO4: now also J14.2 (Pin_2)
- net GPIO5: now reaches U1.34 (IO5)
- net GPIO5: now also J14.3 (Pin_3)
- no-connect marks 6 -> 4
Other:
- moved on the sheet: J4
