File: Hardware/BoverJR/PCBWAY/Wakanda_MultiRobot/Wakanda_MultiRobot/Wakanda_MultiRobot.kicad_sch (KiCad schematic)
At the start: 26 parts, among them J1 Alimentacion, J10 I2C, J14 RANDOM, J2 Conn_01X03, J3 Sensor Distancia 1, J3 TATAMI Frontal Derecho, J4 Conn_01X03, J4 TATAMI Frontal Izquierdo, J5 Conn_01X03, J6 Conn_01X03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

Commit message: mejore y quedo listo para verificar wakanda multi
Parts:
- removed P4: Mounting_Hole, EESTN5:Separador_M3_5mm, symbol 2018---MiniSumo---NANO---DRV8872-rescue:Mounting_Hole-EESTN51
- C10, C9: footprint Capacitor_THT:CP_Axial_L10.0mm_D4.5mm_P15.00mm_Horizontal -> EESTN5:CAP_ELEC_SMD_4X5.5
Changed lines of the file:
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@@
       (effects (font (size 1.016 1.016)) (justify left))
     )
-    (property "Footprint" "Capacitor_THT:CP_Axial_L10.0mm_D4.5mm_P15.00mm_Horizontal" (at 56.134 46.609 0)
+    (property "Footprint" "EESTN5:CAP_ELEC_SMD_4X5.5" (at 56.134 46.609 0)
       (effects (font (size 0.762 0.762)) hide)
     )
@@
         (path "/7706e104-9d42-4651-8ea1-0974927a2230"
           (reference "C10") (unit 1)
-        )
-      )
-    )
-  )
-  (symbol (lib_id "2018---MiniSumo---NANO---DRV8872-rescue:Mounting_Hole-EESTN51") (at 279.019 27.178 0) (unit 1)
-    (in_bom yes) (on_board yes) (dnp no)
-    (property "Reference" "P4" (at 279.019 24.257 0)
-      (effects (font (size 1.27 1.27)))
-    )
-    (property "Value" "Mounting_Hole" (at 279.019 24.003 0)
-      (effects (font (size 1.27 1.27)) hide)
-    )
-    (property "Footprint" "EESTN5:Separador_M3_5mm" (at 279.019 27.178 0)
-      (effects (font (size 1.524 1.524)) hide)
-    )
-    (property "Datasheet" "" (at 279.019 27.178 0)
-      (effects (font (size 1.524 1.524)) hide)
-    )
-    (instances
-      (project "wakanda-board"
-        (path "/19267798-4e4c-4aeb-bec3-b7452995418d"
-          (reference "P4") (unit 1)
-        )
-      )
-      (project "2022-XDecito"
-        (path "/5528bcad-2950-4673-90eb-c37e6952c475"
-          (reference "P3") (unit 1)
-        )
-      )
-      (project "Wakanda_MultiRobot"
-        (path "/7706e104-9d42-4651-8ea1-0974927a2230"
-          (reference "P4") (unit 1)
         )
       )
@@
       (project "Wakanda_MultiRobot"
         (path "/7706e104-9d42-4651-8ea1-0974927a2230"
-          (reference "P1") (unit 1)
+          (reference "P4") (unit 1)
         )
       )
@@
       (effects (font (size 1.016 1.016)) (justify left))
     )
-    (property "Footprint" "Capacitor_THT:CP_Axial_L10.0mm_D4.5mm_P15.00mm_Horizontal" (at 77.47 47.498 0)
+    (property "Footprint" "EESTN5:CAP_ELEC_SMD_4X5.5" (at 77.47 47.498 0)
       (effects (font (size 0.762 0.762)) hide)
     )

Commit message: verifique por 3d , falta ver las vias para pads y eñ gerber y listo
Parts:
- J2, J3, J4, J5, J6: footprint EESTN5:Pin_Header_3 -> EESTN5:Pin_Strip_3
Changed lines of the file:
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@@
       (effects (font (size 1.27 1.27)) (justify left) hide)
     )
-    (property "Footprint" "EESTN5:Pin_Header_3" (at 108.331 113.03 0)
+    (property "Footprint" "EESTN5:Pin_Strip_3" (at 108.331 113.03 0)
       (effects (font (size 1.27 1.27)) hide)
     )
@@
       (effects (font (size 1.27 1.27)) (justify left) hide)
     )
-    (property "Footprint" "EESTN5:Pin_Header_3" (at 82.677 112.903 0)
+    (property "Footprint" "EESTN5:Pin_Strip_3" (at 82.677 112.903 0)
       (effects (font (size 1.27 1.27)) hide)
     )
@@
       (effects (font (size 1.27 1.27)) (justify left) hide)
     )
-    (property "Footprint" "EESTN5:Pin_Header_3" (at 108.204 133.35 0)
+    (property "Footprint" "EESTN5:Pin_Strip_3" (at 108.204 133.35 0)
       (effects (font (size 1.27 1.27)) hide)
     )
@@
       (effects (font (size 1.27 1.27)))
     )
-    (property "Footprint" "EESTN5:Pin_Header_3" (at 145.161 113.538 0)
+    (property "Footprint" "EESTN5:Pin_Strip_3" (at 145.161 113.538 0)
       (effects (font (size 1.27 1.27)) hide)
     )
@@
       (effects (font (size 1.27 1.27)))
     )
-    (property "Footprint" "EESTN5:Pin_Header_3" (at 145.034 94.488 0)
+    (property "Footprint" "EESTN5:Pin_Strip_3" (at 145.034 94.488 0)
       (effects (font (size 1.27 1.27)) hide)
     )
@@
       (effects (font (size 1.27 1.27)) (justify left) hide)
     )
-    (property "Footprint" "EESTN5:Pin_Header_3" (at 108.331 95.758 0)
+    (property "Footprint" "EESTN5:Pin_Strip_3" (at 108.331 95.758 0)
       (effects (font (size 1.27 1.27)) hide)
     )
@@
       (effects (font (size 1.27 1.27)) (justify left) hide)
     )
-    (property "Footprint" "EESTN5:Pin_Header_3" (at 82.677 95.631 0)
-      (effects (font (size 1.27 1.27)) hide)
-    )
+    (property "Footprint" "EESTN5:Pin_Strip_3" (at 82.677 95.631 0)
+      (effects (font (size 1.27 1.27)) hide)
+    )

Commit message: corregi placa wakanda segun buistos
Parts:
- J1: footprint EESTN5:BORNERA3_AZUL -> EESTN5-v2:BORNERA3_AZUL_VIAS
Changed lines of the file:
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@@
       (effects (font (size 1.524 1.524)))
     )
-    (property "Footprint" "EESTN5:BORNERA3_AZUL" (at 18.923 36.83 0)
+    (property "Footprint" "EESTN5-v2:BORNERA3_AZUL_VIAS" (at 18.923 36.83 0)
       (effects (font (size 1.524 1.524)) hide)
     )

Commit message: cambios a wakanda en pcb
Other:
- moved on the sheet: C10, C9
Changed lines of the file:
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@@
   (junction (at 175.26 42.672) (diameter 0) (color 0 0 0 0)
   )
-  (junction (at 53.594 35.179) (diameter 0) (color 0 0 0 0)
-  )
   (junction (at 156.464 42.672) (diameter 0) (color 0 0 0 0)
   )
   (junction (at 63.754 50.419) (diameter 0) (color 0 0 0 0)
   )
+  (junction (at 45.7454 35.179) (diameter 0) (color 0 0 0 0)
+  )
   (junction (at 208.915 28.194) (diameter 0) (color 0 0 0 0)
   )
@@
   (junction (at 216.027 21.336) (diameter 0) (color 0 0 0 0)
   )
+  (junction (at 87.7316 35.179) (diameter 0) (color 0 0 0 0)
+  )
+  (junction (at 63.754 50.3174) (diameter 0) (color 0 0 0 0)
+  )
   (junction (at 187.96 42.037) (diameter 0) (color 0 0 0 0)
   )
@@
     (stroke (width 0) (type default))
   )
+  (wire (pts (xy 63.754 50.3174) (xy 63.754 50.419))
+    (stroke (width 0) (type default))
+  )
   (wire (pts (xy 91.186 130.81) (xy 103.124 130.81))
     (stroke (width 0) (type default))
@@
     (stroke (width 0) (type default))
   )
+  (wire (pts (xy 87.7316 35.0774) (xy 87.7316 35.179))
+    (stroke (width 0) (type default))
+  )
   (wire (pts (xy 91.313 93.218) (xy 103.251 93.218))
     (stroke (width 0) (type default))
@@
     (stroke (width 0) (type default))
   )
-  (wire (pts (xy 53.594 47.879) (xy 53.594 50.419))
+  (wire (pts (xy 45.7454 48.133) (xy 45.7454 50.419))
     (stroke (width 0) (type default))
   )
@@
     (stroke (width 0) (type default))
   )
-  (wire (pts (xy 53.594 50.419) (xy 63.754 50.419))
+  (wire (pts (xy 45.7454 50.419) (xy 63.754 50.419))
     (stroke (width 0) (type default))
   )
@@
     (stroke (width 0) (type default))
   )
+  (wire (pts (xy 87.7316 35.179) (xy 87.7316 38.5064))
+    (stroke (width 0) (type default))
+  )
   (wire (pts (xy 91.313 110.49) (xy 103.251 110.49))
     (stroke (width 0) (type default))
@@
     (stroke (width 0) (type default))
   )
-  (wire (pts (xy 45.339 35.179) (xy 53.594 35.179))
+  (wire (pts (xy 45.339 35.179) (xy 45.7454 35.179))
     (stroke (width 0) (type default))
   )
@@
     (stroke (width 0) (type default))
   )
-  (wire (pts (xy 53.594 37.719) (xy 53.594 35.179))
+  (wire (pts (xy 45.7454 37.973) (xy 45.7454 35.179))
     (stroke (width 0) (type default))
   )
@@
     (stroke (width 0) (type default))
   )
-  (wire (pts (xy 63.754 42.799) (xy 63.754 50.419))
+  (wire (pts (xy 63.754 42.799) (xy 63.754 50.3174))
     (stroke (width 0) (type default))
   )
@@
     (stroke (width 0) (type default))
   )
-  (wire (pts (xy 74.93 48.768) (xy 74.93 50.419))
+  (wire (pts (xy 87.7316 48.6664) (xy 87.7316 50.3174))
     (stroke (width 0) (type default))
   )
@@
     (stroke (width 0) (type default))
   )
-  (wire (pts (xy 63.754 50.419) (xy 74.93 50.419))
+  (wire (pts (xy 63.754 50.3174) (xy 87.7316 50.3174))
     (stroke (width 0) (type default))
   )
@@
     (stroke (width 0) (type default))
   )
-  (wire (pts (xy 53.594 35.179) (xy 56.134 35.179))
+  (wire (pts (xy 45.7454 35.179) (xy 56.134 35.179))
     (stroke (width 0) (type default))
   )
@@
     (stroke (width 0) (type default))
   )
-  (wire (pts (xy 74.93 35.179) (xy 74.93 38.608))
-    (stroke (width 0) (type default))
-  )
   (wire (pts (xy 156.464 41.402) (xy 156.464 42.672))
     (stroke (width 0) (type default))
@@
     (stroke (width 0) (type default))
   )
+  (wire (pts (xy 87.7316 35.179) (xy 74.93 35.179))
+    (stroke (width 0) (type default))
+  )
   (polyline (pts (xy 200.152 110.617) (xy 200.152 110.871))
     (stroke (width 0) (type default))
@@
     )
   )
-  (symbol (lib_id "EESTN5:CAPAPOL") (at 53.594 42.799 0) (unit 1)
+  (symbol (lib_id "EESTN5:CAPAPOL") (at 45.7454 43.053 0) (unit 1)
     (in_bom yes) (on_board yes) (dnp no) (fields_autoplaced)
-    (property "Reference" "C10" (at 57.15 42.164 0)
+    (property "Reference" "C10" (at 49.3014 42.418 0)
       (effects (font (size 1.016 1.016)) (justify left))
     )
-    (property "Value" "10uF" (at 57.15 44.704 0)
+    (property "Value" "10uF" (at 49.3014 44.958 0)
       (effects (font (size 1.016 1.016)) (justify left))
     )
-    (property "Footprint" "EESTN5:CAP_ELEC_SMD_4X5.5" (at 56.134 46.609 0)
+    (property "Footprint" "EESTN5:CAP_ELEC_SMD_4X5.5" (at 48.2854 46.863 0)
       (effects (font (size 0.762 0.762)) hide)
     )
-    (property "Datasheet" "" (at 53.594 42.799 0)
+    (property "Datasheet" "" (at 45.7454 43.053 0)
       (effects (font (size 7.62 7.62)))
     )
@@
     )
   )
-  (symbol (lib_id "EESTN5:CAPAPOL") (at 74.93 43.688 0) (unit 1)
+  (symbol (lib_id "EESTN5:CAPAPOL") (at 87.7316 43.5864 0) (unit 1)
     (in_bom yes) (on_board yes) (dnp no) (fields_autoplaced)
-    (property "Reference" "C9" (at 78.74 43.053 0)
+    (property "Reference" "C9" (at 91.5416 42.9514 0)
       (effects (font (size 1.016 1.016)) (justify left))
     )
-    (property "Value" "100uF" (at 78.74 45.593 0)
+    (property "Value" "100uF" (at 91.5416 45.4914 0)
       (effects (font (size 1.016 1.016)) (justify left))
     )
-    (property "Footprint" "EESTN5:CAP_ELEC_SMD_4X5.5" (at 77.47 47.498 0)
+    (property "Footprint" "EESTN5:CAP_ELEC_SMD_4X5.5" (at 90.2716 47.3964 0)
       (effects (font (size 0.762 0.762)) hide)
     )
-    (property "Datasheet" "" (at 74.93 43.688 0)
+    (property "Datasheet" "" (at 87.7316 43.5864 0)
       (effects (font (size 7.62 7.62)))
     )

Commit message: agrego cambios de gerber antes de fabricar que colgue
Parts:
- J1: footprint EESTN5-v2:BORNERA3_AZUL_VIAS -> EESTN5:BORNERA3_AZUL_VIAS
- J3: value TATAMI Frontal Derecho -> ~
Connections:
- net +5V: now also J3.1 (P1), J4.1 (P1), J5.2 (P2), J6.2 (P2), SW1.3 (P3); no longer J3.2 (P2), J4.2 (P2), J5.1 (P1), J6.1 (P1), SW1.2 (P2)
- net GND: now also J3.2 (P2), J4.2 (P2), J5.1 (P1), J6.1 (P1); no longer J3.1 (P1), J4.1 (P1), J5.2 (P2), J6.2 (P2)
- net SENSOR5: now also U1.11 (IO35); no longer U1.10 (IO34)
- net START: now also SW1.2 (P2), U1.10 (IO34); no longer SW1.3 (P3), U1.11 (IO35)
- net TATAMI_FD renamed SENSOR6
- net SENSOR6: now also J4.3 (P3); no longer J3.3 (P3)
- net TATAMI_FI renamed SENSOR7
- net SENSOR7: now also J3.3 (P3); no longer J4.3 (P3)
Other:
- note added: "SENSORES DE DISTANCIA Y LINEA:"
- note removed: "SENSORES DE DISTANCIA:"
- note removed: "SENSORES DE LÍNEA:"
- moved on the sheet: J3, J4, J6
