File: Hardware/BoverJR/PCBWAY/Wakanda_MultiRobot/Wakanda_MultiRobot/Driver_motores.kicad_sch (KiCad schematic)
At the start: 11 parts, among them J10 M2, J9 M1, U2 DRV8872, U3 DRV8872

Commit message: sch de driver modificado
Parts:
- removed J9: M1, EESTN5:BORNERA3_AZUL, symbol 2018---MiniSumo---NANO---DRV8872-rescue:TB_1X3-EESTN51
- added J10: M2, EESTN5:BORNERA2_AZUL, symbol 2018---MiniSumo---NANO---DRV8872-rescue:TB_1X2-EESTN51
- U2: value DRV8872 -> TB67H451AFNG
Connections:
- net at U2.6 (OUT1): now also J10.2
- net at U2.8 (OUT2): now also J10.1

Commit message: ordene PCB
Parts:
- C1, C2: footprint EESTN5:C_1206 -> EESTN5:C_0805
- J10: value M2 -> M1

Commit message: casi termino PCB
Parts:
- removed R1, R2: Risen, EESTN5:PTC_1210, symbol 2018---MiniSumo---NANO---DRV8872-rescue:R-EESTN51
- removed U3: DRV8872, EESTN5:SSOP-8, symbol 2018---MiniSumo---NANO---DRV8872-rescue:DRV8872-EESTN51
- added U2: TB67H451AFNG, EESTN5:SSOP-8, symbol 2018---MiniSumo---NANO---DRV8872-rescue:DRV8872-EESTN51
Connections:
- net GND: now also U2.7 (RS), U2.1 (GND), U2.7 (RS)
- net M2A: now also U2.3 (IN1)
- net M2B: now also U2.2 (IN2)
- net Vin: now also U2.5 (VM)
- net +5V: now reaches U2.4 (VREF)
- net +5V: now also U2.4 (VREF)
- net at J10.2: now also U2.6 (OUT1)
- net at J10.1: now also U2.8 (OUT2)
- no-connect marks 2 -> 0
Other:
- moved on the sheet: LOGO1

Commit message: placa casi terminada falta 3d y estetica
Parts:
- J10: value M2 -> M1
Connections:
- net at U2.6 (OUT1): now also J10.1; no longer J10.2 (x2)
- net at U2.8 (OUT2): now also J10.2; no longer J10.1 (x2)
Changed lines of the file:
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@@
     )
   )
-  (symbol (lib_id "2018---MiniSumo---NANO---DRV8872-rescue:TB_1X2-EESTN51") (at 164.465 43.815 0) (mirror y) (unit 1)
+  (symbol (lib_name "TB_1X2-EESTN51_1") (lib_id "2018---MiniSumo---NANO---DRV8872-rescue:TB_1X2-EESTN51") (at 164.465 43.815 0) (mirror y) (unit 1)
     (in_bom yes) (on_board yes) (dnp no)
     (property "Reference" "J10" (at 164.465 36.195 0)
       (effects (font (size 1.524 1.524)))
     )
-    (property "Value" "M1" (at 163.068 51.308 0)
-      (effects (font (size 1.524 1.524)))
-    )
-    (property "Footprint" "EESTN5:BORNERA2_AZUL" (at 165.735 42.545 0)
-      (effects (font (size 1.524 1.524)) hide)
-    )
-    (property "Datasheet" "" (at 165.735 42.545 0)
+    (property "Value" "M1" (at 165.862 51.308 0)
+      (effects (font (size 1.524 1.524)))
+    )
+    (property "Footprint" "EESTN5:BORNERA2_AZUL" (at 163.195 42.545 0)
+      (effects (font (size 1.524 1.524)) hide)
+    )
+    (property "Datasheet" "" (at 163.195 42.545 0)
       (effects (font (size 1.524 1.524)))
     )
@@
     )
   )
-  (symbol (lib_id "2018---MiniSumo---NANO---DRV8872-rescue:TB_1X2-EESTN51") (at 164.465 81.915 0) (mirror y) (unit 1)
-    (in_bom yes) (on_board yes) (dnp no)
-    (property "Reference" "J10" (at 164.465 74.295 0)
-      (effects (font (size 1.524 1.524)))
-    )
-    (property "Value" "M2" (at 163.068 89.408 0)
-      (effects (font (size 1.524 1.524)))
-    )
-    (property "Footprint" "EESTN5:BORNERA2_AZUL" (at 165.735 80.645 0)
-      (effects (font (size 1.524 1.524)) hide)
-    )
-    (property "Datasheet" "" (at 165.735 80.645 0)
-      (effects (font (size 1.524 1.524)))
-    )
-    (pin "1")
-    (pin "2")
-    (instances
-      (project "2023-wakanda-V1"
-        (path "/19267798-4e4c-4aeb-bec3-b7452995418d/f8226101-1b75-4d42-8152-d386adfd0d30"
-          (reference "J10") (unit 1)
-        )
-      )
-      (project "2022-XDecito"
-        (path "/5528bcad-2950-4673-90eb-c37e6952c475/00000000-0000-0000-0000-00005b0f2c2d"
-          (reference "J13") (unit 1)
-        )
-      )
-      (project "Driver_motores"
-        (path "/7669a348-9f1c-4f34-9714-a6db73698347"
-          (reference "J10") (unit 1)
-        )
-      )
-      (project "Wakanda_MultiRobot"
-        (path "/7706e104-9d42-4651-8ea1-0974927a2230/0a488edf-d039-4a58-8e18-6b013530cf76"
-          (reference "J12") (unit 1)
-        )
-      )
-    )
-  )
   (symbol (lib_id "2018---MiniSumo---NANO---DRV8872-rescue:C-EESTN51") (at 125.095 55.245 0) (unit 1)
     (in_bom yes) (on_board yes) (dnp no)
@@
         )
       )
+    )
+  )
+  (symbol (lib_name "TB_1X2-EESTN51_1") (lib_id "2018---MiniSumo---NANO---DRV8872-rescue:TB_1X2-EESTN51") (at 164.465 81.915 0) (mirror y) (unit 1)
+    (in_bom yes) (on_board yes) (dnp no)
+    (property "Reference" "J10" (at 164.465 74.295 0)
+      (effects (font (size 1.524 1.524)))
+    )
+    (property "Value" "M1" (at 165.862 89.408 0)
+      (effects (font (size 1.524 1.524)))
+    )
+    (property "Footprint" "EESTN5:BORNERA2_AZUL" (at 163.195 80.645 0)
+      (effects (font (size 1.524 1.524)) hide)
+    )
+    (property "Datasheet" "" (at 163.195 80.645 0)
+      (effects (font (size 1.524 1.524)))
+    )
+    (pin "1")
+    (pin "2")
+    (instances
+      (project "2023-wakanda-V1"
+        (path "/19267798-4e4c-4aeb-bec3-b7452995418d/f8226101-1b75-4d42-8152-d386adfd0d30"
+          (reference "J10") (unit 1)
+        )
+      )
+      (project "2022-XDecito"
+        (path "/5528bcad-2950-4673-90eb-c37e6952c475/00000000-0000-0000-0000-00005b0f2c2d"
+          (reference "J13") (unit 1)
+        )
+      )
+      (project "Driver_motores"
+        (path "/7669a348-9f1c-4f34-9714-a6db73698347"
+          (reference "J1") (unit 1)
+        )
+      )
+      (project "Wakanda_MultiRobot"
+        (path "/7706e104-9d42-4651-8ea1-0974927a2230/0a488edf-d039-4a58-8e18-6b013530cf76"
+          (reference "J12") (unit 1)
+        )
+      )

Commit message: verifique por 3d
Parts:
- J10: value M1 -> M2
Changed lines of the file:
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@@
       (effects (font (size 1.524 1.524)))
     )
-    (property "Value" "M1" (at 165.862 89.408 0)
+    (property "Value" "M2" (at 165.862 89.408 0)
       (effects (font (size 1.524 1.524)))
     )

Commit message: recomendacion de bustos
Parts:
- C3: footprint EESTN5:CAP_ELEC_10X8mm -> EESTN5:CAP_ELEC_5x11mm
Changed lines of the file:
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@@
       (effects (font (size 1.016 1.016)) (justify left))
     )
-    (property "Footprint" "EESTN5:CAP_ELEC_10X8mm" (at 133.985 59.055 0)
+    (property "Footprint" "EESTN5:CAP_ELEC_5x11mm" (at 133.985 59.055 0)
       (effects (font (size 0.762 0.762)) hide)
     )

Commit message: mejore y quedo listo para verificar wakanda multi
Parts:
- removed LOGO1: Mounting_Hole, EESTN5:LOGO_EESTN5, symbol 2018---MiniSumo---NANO---DRV8872-rescue:Mounting_Hole-EESTN51
Changed lines of the file:
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@@
-    )
-  )
-  (symbol (lib_id "2018---MiniSumo---NANO---DRV8872-rescue:Mounting_Hole-EESTN51") (at 97.028 102.235 0) (unit 1)
-    (in_bom yes) (on_board yes) (dnp no)
-    (property "Reference" "LOGO1" (at 97.028 97.155 0)
-      (effects (font (size 1.27 1.27)))
-    )
-    (property "Value" "Mounting_Hole" (at 97.028 99.06 0)
-      (effects (font (size 1.27 1.27)) hide)
-    )
-    (property "Footprint" "EESTN5:LOGO_EESTN5" (at 97.028 102.235 0)
-      (effects (font (size 1.524 1.524)) hide)
-    )
-    (property "Datasheet" "" (at 97.028 102.235 0)
-      (effects (font (size 1.524 1.524)) hide)
-    )
-    (instances
-      (project "2023-wakanda-V1"
-        (path "/19267798-4e4c-4aeb-bec3-b7452995418d/f8226101-1b75-4d42-8152-d386adfd0d30"
-          (reference "LOGO1") (unit 1)
-        )
-      )
-      (project "2022-XDecito"
-        (path "/5528bcad-2950-4673-90eb-c37e6952c475/00000000-0000-0000-0000-00005b0f2c2d"
-          (reference "LOGO1") (unit 1)
-        )
-      )
-      (project "Driver_motores"
-        (path "/7669a348-9f1c-4f34-9714-a6db73698347"
-          (reference "LOGO1") (unit 1)
-        )
-      )
-      (project "Wakanda_MultiRobot"
-        (path "/7706e104-9d42-4651-8ea1-0974927a2230/0a488edf-d039-4a58-8e18-6b013530cf76"
-          (reference "LOGO1") (unit 1)
-        )
-      )
     )
   )
