File: Hardware/BoverJR/PCBWAY/Wakanda_MultiRobot/Wakanda_MultiRobot/Driver_motores.kicad_sch (KiCad schematic)
At the start: 8 parts, among them J10 M1, J10 M2, U2 TB67H451AFNG

Commit message: corregi placa wakanda segun buistos
Parts:
- J10: footprint EESTN5:BORNERA2_AZUL -> EESTN5-v2:BORNERA2_AZUL_VIAS
Changed lines of the file:
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@@
       (effects (font (size 1.524 1.524)))
     )
-    (property "Footprint" "EESTN5:BORNERA2_AZUL" (at 163.195 80.645 0)
+    (property "Footprint" "EESTN5-v2:BORNERA2_AZUL_VIAS" (at 163.195 80.645 0)
       (effects (font (size 1.524 1.524)) hide)
     )

Commit message: agregue pads a ic tb67
Parts:
- U2: footprint EESTN5:SSOP-8 -> EESTN5-v2:SSOP-8_disipa
Changed lines of the file:
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@@
       (effects (font (size 1.524 1.524)))
     )
-    (property "Footprint" "EESTN5:SSOP-8" (at 107.315 51.435 0)
+    (property "Footprint" "EESTN5-v2:SSOP-8_disipa" (at 107.315 51.435 0)
       (effects (font (size 1.524 1.524)) hide)
     )
@@
       (effects (font (size 1.524 1.524)))
     )
-    (property "Footprint" "EESTN5:SSOP-8" (at 107.315 89.535 0)
+    (property "Footprint" "EESTN5-v2:SSOP-8_disipa" (at 107.315 89.535 0)
       (effects (font (size 1.524 1.524)) hide)
     )

Commit message: esperando verificacion de pcbway ya cargue 6 gerber
Parts:
- J10: footprint EESTN5:BORNERA2_AZUL -> EESTN5:BORNERA2_AZUL_VIAS
- J10: footprint EESTN5-v2:BORNERA2_AZUL_VIAS -> EESTN5:BORNERA2_AZUL_VIAS
Changed lines of the file:
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@@
       (effects (font (size 1.524 1.524)))
     )
-    (property "Footprint" "EESTN5:BORNERA2_AZUL" (at 163.195 42.545 0)
+    (property "Footprint" "EESTN5:BORNERA2_AZUL_VIAS" (at 163.195 42.545 0)
       (effects (font (size 1.524 1.524)) hide)
     )
@@
       (effects (font (size 1.524 1.524)))
     )
-    (property "Footprint" "EESTN5-v2:BORNERA2_AZUL_VIAS" (at 163.195 80.645 0)
+    (property "Footprint" "EESTN5:BORNERA2_AZUL_VIAS" (at 163.195 80.645 0)
       (effects (font (size 1.524 1.524)) hide)
     )
