File: Hardware/BoverJR/PCBWAY/Wakanda_MultiRobot/Wakanda_MultiRobot/Wakanda_MultiRobot.kicad_pcb (KiCad board)
At the start: 2 copper layers, 50 x 50 mm, 33 parts, among them J1 TATAMI Frontal Derecho, J10 Conn_01X03, J11 M1, J12 Alimentacion, J13 M2, J2 Sensor Distancia 1, J3 TATAMI Frontal Izquierdo, J4 Conn_01X03, J5 Conn_01X03, J6 Conn_01X03, J7 Programador, J8 I2C, J9 RANDOM, P1 Mounting_Hole, P2 Mounting_Hole, P3 Mounting_Hole, SW1 START, U1 ESP32-WROOM-32E, U2 TB67H451AFNG, U3 TB67H451AFNG, U4 AMS1117-3.3

Commit message: verifique por 3d , falta ver las vias para pads y eñ gerber y listo
Parts:
- removed the C2 at (162.1, 84.5)
- removed C5: 100uF 35V, EESTN5:CAP_ELEC_5x11mm
- removed C6: 100uF, EESTN5:CAP_ELEC_SMD_4X5.5
- removed the J9 at (184.5, 85.5)
- added C10: 10uF, EESTN5:CAP_ELEC_SMD_4X5.5, F.Cu at (182.8, 92.9)
- added C3: 100uF 35V, EESTN5:CAP_ELEC_5x11mm, F.Cu at (153.1, 91.6)
- added C9: 100uF, EESTN5:CAP_ELEC_SMD_4X5.5, F.Cu at (169.6, 93.3)
- added J14: RANDOM, EESTN5:pin_strip_4, F.Cu at (184.2, 85.4)
- C7: value 10uF -> 100nF; footprint EESTN5:CAP_ELEC_SMD_4X5.5 -> EESTN5:C_0805
- J2: renamed from J5; footprint EESTN5:Pin_Header_3 -> EESTN5:Pin_Strip_3
- J3: renamed from J2; footprint EESTN5:Pin_Header_3 -> EESTN5:Pin_Strip_3
- J4: footprint EESTN5:Pin_Header_3 -> EESTN5:Pin_Strip_3
- J5: renamed from J6; footprint EESTN5:Pin_Header_3 -> EESTN5:Pin_Strip_3
- J6: renamed from J10; footprint EESTN5:Pin_Header_3 -> EESTN5:Pin_Strip_3
- J7: renamed from J1; footprint EESTN5:Pin_Header_3 -> EESTN5:Pin_Strip_3
- J8: renamed from J3; footprint EESTN5:Pin_Header_3 -> EESTN5:Pin_Strip_3
- moved C7 22.3 mm to (162.1, 84.7), turned to 90 degrees
- moved P4 0.50 mm to (143.4, 63.3)
- renumbered C4 to C1, C3 to C2, C1 to C8, J12 to J1, J8 to J10, J13 to J12, J7 to J9, P1 to P4, R1 to R3, R2 to R4, U3 to U2, U2 to U3
Connections:
- C7 pad 1: +5V -> /EN
Routing:
- net /SENSOR4: track 12.8 -> 9.05 mm
- net /SENSOR3: track 13.6 -> 9.87 mm
- net /M_DER_B: track 25.7 -> 28.8 mm
- net /M_DER_A: track 25.7 -> 28.8 mm
- net /SCL: track 28.3 -> 26.2 mm
- net +3V3: track 71.5 -> 69.7 mm, vias 1 -> 0
- net Net-(U3-OUT2): track 27.5 -> 29.3 mm
- net +5V: track 135.1 -> 136.1 mm, vias 3 -> 2
- net Net-(U3-OUT1): track 26.4 -> 27.2 mm
- net Net-(U2-OUT1): track 9.47 -> 10.3 mm
- net Net-(U2-OUT2): track 9.39 -> 10.2 mm
- net /GPIO5: track 21.3 -> 21.8 mm
- net GND: vias 2 -> 0

Commit message: corregi placa wakanda segun buistos
Parts:
- J1: footprint EESTN5:BORNERA3_AZUL -> EESTN5-v2:BORNERA3_AZUL_VIAS
- J12: footprint EESTN5:BORNERA2_AZUL -> EESTN5-v2:BORNERA2_AZUL_VIAS
- moved C1 4.94 mm to (141.2, 93.6), turned to -90 degrees
- moved P3 0.91 mm to (186.8, 97.2)
- moved P2 0.79 mm to (152.8, 97.3)
- moved U2 0.57 mm to (145.2, 93.6)
- moved J1 0.33 mm to (165.3, 106.3)
- moved J12 0.13 mm to (184.8, 106.3)
- renumbered BOOT1 to BOOT, EN1 to EN
Routing:
- net +5V: track 136.1 -> 145.4 mm
- net Vin: track 36.1 -> 40.6 mm, vias 0 -> 1
- net Net-(U3-OUT1): track 27.2 -> 25.3 mm
- net /SENSOR2: track 17.2 -> 18.8 mm
- net Net-(U3-OUT2): track 29.3 -> 30.7 mm
- net GND: track 4.66 -> 3.28 mm
- net /M_IZQ_A: track 25.7 -> 24.4 mm
- added copper zone on B.Cu, net +5V
- added copper zone on F.Cu, net Net-(U2-OUT1)
- added copper zone on F.Cu, net Net-(U2-OUT2)
- added copper zone on F.Cu, net Net-(U3-OUT1)
- added copper zone on F.Cu, net Net-(U3-OUT2)
- added copper zone on F.Cu, net Vin
