File: Hardware/BoverJR/PCBWAY/PCB art/messi/messi_v1.kicad_sch (KiCad schematic)
At the start: 3 parts

Commit message: agregue a maradoooooooooo
Parts:
- added H4: Mounting_Hole, EESTN5:maradov1_bcu, symbol EESTN5:Mounting_Hole
Changed lines of the file:
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@@
+    )
+  )
+  (symbol (lib_id "EESTN5:Mounting_Hole") (at 144.399 91.44 0) (unit 1)
+    (in_bom yes) (on_board yes) (dnp no) (fields_autoplaced)
+    (property "Reference" "H4" (at 147.32 92.075 0)
+      (effects (font (size 1.27 1.27)) (justify left))
+    )
+    (property "Value" "Mounting_Hole" (at 144.399 88.265 0)
+      (effects (font (size 1.27 1.27)) hide)
+    )
+    (property "Footprint" "EESTN5:maradov1_bcu" (at 144.399 91.44 0)
+      (effects (font (size 1.524 1.524)) hide)
+    )
+    (property "Datasheet" "" (at 144.399 91.44 0)
+      (effects (font (size 1.524 1.524)) hide)
+    )
+    (instances
+      (project "messi_v1"
+        (path "/1156a248-667a-47ac-b655-16a5991e6b18"
+          (reference "H4") (unit 1)
+        )
+      )
     )
   )

Commit message: terrmine llavero messi
Parts:
- added H5: Mounting_Hole, EESTN5:afa_mm, symbol EESTN5:Mounting_Hole
- added H6: Mounting_Hole, EESTN5:bover_mm, symbol EESTN5:Mounting_Hole
- H2: footprint EESTN5:logo_messiv3 -> EESTN5:messi
Changed lines of the file:
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@@
+    )
+  )
+  (symbol (lib_id "EESTN5:Mounting_Hole") (at 144.526 102.997 0) (unit 1)
+    (in_bom yes) (on_board yes) (dnp no) (fields_autoplaced)
+    (property "Reference" "H6" (at 147.447 103.632 0)
+      (effects (font (size 1.27 1.27)) (justify left))
+    )
+    (property "Value" "Mounting_Hole" (at 144.526 99.822 0)
+      (effects (font (size 1.27 1.27)) hide)
+    )
+    (property "Footprint" "EESTN5:bover_mm" (at 144.526 102.997 0)
+      (effects (font (size 1.524 1.524)) hide)
+    )
+    (property "Datasheet" "" (at 144.526 102.997 0)
+      (effects (font (size 1.524 1.524)) hide)
+    )
+    (instances
+      (project "messi_v1"
+        (path "/1156a248-667a-47ac-b655-16a5991e6b18"
+          (reference "H6") (unit 1)
+        )
+      )
     )
   )
@@
       (effects (font (size 1.27 1.27)) hide)
     )
-    (property "Footprint" "EESTN5:logo_messiv3" (at 144.399 80.518 0)
+    (property "Footprint" "EESTN5:messi" (at 144.399 80.518 0)
       (effects (font (size 1.524 1.524)) hide)
     )
@@
         )
       )
+    )
+  )
+  (symbol (lib_id "EESTN5:Mounting_Hole") (at 144.526 97.282 0) (unit 1)
+    (in_bom yes) (on_board yes) (dnp no) (fields_autoplaced)
+    (property "Reference" "H5" (at 147.447 97.917 0)
+      (effects (font (size 1.27 1.27)) (justify left))
+    )
+    (property "Value" "Mounting_Hole" (at 144.526 94.107 0)
+      (effects (font (size 1.27 1.27)) hide)
+    )
+    (property "Footprint" "EESTN5:afa_mm" (at 144.526 97.282 0)
+      (effects (font (size 1.524 1.524)) hide)
+    )
+    (property "Datasheet" "" (at 144.526 97.282 0)
+      (effects (font (size 1.524 1.524)) hide)
+    )
+    (instances
+      (project "messi_v1"
+        (path "/1156a248-667a-47ac-b655-16a5991e6b18"
+          (reference "H5") (unit 1)
+        )
+      )
