File: Hardware/BoverJR/PCBWAY/Driver_TB67H451AFNG/Driver_TB67H451AFNG.kicad_sch (KiCad schematic)
At the start: 8 parts, among them J10 M2, J10 TB_1X2, J4 Conn_01x04_Pin, U2 TB67H451AFNG

Commit message: Rediseño Driver TB67
Parts:
- J10: footprint EESTN5-v2:BORNERA2_AZUL -> EESTN5-v2:BORNERA2_AZUL_HOLES+
- U2: footprint EESTN5-v2:SSOP-8 -> EESTN5-v2:SSOP-8_disipa
Changed lines of the file:
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@@
       (effects (font (size 1.524 1.524)))
     )
-    (property "Footprint" "EESTN5-v2:SSOP-8" (at 113.919 113.1062 0)
+    (property "Footprint" "EESTN5-v2:SSOP-8_disipa" (at 113.919 113.1062 0)
       (effects (font (size 1.524 1.524)) hide)
     )
@@
       (effects (font (size 1.524 1.524)))
     )
-    (property "Footprint" "EESTN5-v2:BORNERA2_AZUL" (at 167.3352 104.2162 0)
+    (property "Footprint" "EESTN5-v2:BORNERA2_AZUL_HOLES+" (at 167.3352 104.2162 0)
       (effects (font (size 1.524 1.524)) hide)
     )
