File: Hardware/BoverJR/PCBWAY/sensores/qre1113/qre1113_modulo/qre1113_modulo.kicad_sch (KiCad schematic)
At the start: 4 parts, among them J1 qre1113_out, U1 QRE1113

Commit message: Terminada placa qre1113
Parts:
- removed R1: 10k, symbol EESTN5:R
- removed R2: 220, symbol EESTN5:R
- removed U1: QRE1113, QRE1113GR, symbol EESTN5:QRE1113
- added H1: HOLE, EESTN5-v2:Separador_M3_5mm, symbol Mechanical:MountingHole
- added R16: 4k7, EESTN5-v2:R_0805, symbol Device:R
- added R6: 100, EESTN5-v2:R_0805, symbol Device:R
- added U1: QRE1113GR, OptoDevice:OnSemi_CASE100CY, symbol Sensor_Proximity:QRE1113GR
- J1: footprint (none) -> Connector_PinHeader_2.54mm:PinHeader_1x03_P2.54mm_Vertical
Connections:
- net GND: now also J1.2 (P2), U1.2 (K), U1.4; no longer J1.3 (P3)
- net +5V renamed +3V3
- net +3V3: now also R16.2, R6.1
- new net: R6.2, U1.1 (A)
- new net OUT: J1.3 (P3), R16.1, U1.3
Other:
- title: (none) -> QRE-1113
- moved on the sheet: J1
