File: Hardware/BoverJR/PCBWAY/qre1113/qre1113_modulo/qre1113_modulo.kicad_pcb (KiCad board)
At the start: 2 copper layers, 12 x 9 mm, 5 parts, among them J1 qre1113_out, U1 QRE1113GR

Commit message: agrego cambios de gerber antes de fabricar que colgue
Changed lines of the file:
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@@
     (pcbplotparams
       (layerselection 0x00010fc_ffffffff)
-      (plot_on_all_layers_selection 0x0000000_00000000)
+      (plot_on_all_layers_selection 0x0001000_00000000)
       (disableapertmacros false)
       (usegerberextensions false)
@@
       (psa4output false)
       (plotreference true)
-      (plotvalue true)
+      (plotvalue false)
       (plotinvisibletext false)
       (sketchpadsonfab false)
@@
       (outputformat 1)
       (mirror false)
-      (drillshape 1)
+      (drillshape 0)
       (scaleselection 1)
-      (outputdirectory "")
+      (outputdirectory "../../gerber/QREX1/")
     )
   )
@@
         (effects (font (size 1.524 1.524) (thickness 0.3048)))
     )
-    (pad "1" thru_hole circle (at 0 0 180) (size 3.25 3.25) (drill 3.25) (layers "*.Cu" "F.SilkS"))
+    (pad "1" thru_hole circle (at 0 0 180) (size 3.25 3.25) (drill 3.25) (layers "*.Cu" "*.Mask"))
     (model "D:/APPS Mauri/KiCad Carpetas/EESTN5 - Librerias Kicad/EESTN5.3dshapes/Separador_M3_5mm.wrl"
       (offset (xyz 0 0 0))
@@
     )
   )
-  (gr_rect (start 131.192832 120.47) (end 119.192832 129.47)
+  (gr_rect (start 119.192832 120.47) (end 131.192832 129.47)
     (stroke (width 0.1) (type default)) (fill none) (layer "Edge.Cuts"))
   (gr_text "+" (at 127.09 123.1325) (layer "F.SilkS")
